File: external-ethernet.kicad_sch (KiCad schematic)
At the start: 29 parts, among them IC24 ENC28J60-I_SO, J6 SS-60300-103, T1 PT61017XPEL, Y1 25MHz

Commit message: first round of revisions
Parts:
- FB7: renamed from L3; value 60R 80mA -> BLM02PX600SN1D; symbol SamacSys_Parts:74279260 -> Oro:FerriteBead
- renumbered R18 to R19, R19 to R20, R20 to R21, R21 to R22, R22 to R23, R23 to R24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
