File: iscp-pad.kicad_sch (KiCad schematic)
At the start: 6 parts, among them J6 OroConn6p

Commit message: first round of revisions
Parts:
- renumbered R17 to R18
Changed lines of the file:
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@@
         )
         (path "/e89dcd22-1250-4a5b-b778-1c95a0dd623d/259c9346-7ad9-40c3-9e14-9b19afc78ddf"
-          (reference "R16") (unit 1)
+          (reference "R17") (unit 1)
         )
       )
@@
   (symbol (lib_id "SamacSys_Parts:CRGP2512F1K0") (at 124.46 81.28 90) (unit 1)
     (in_bom yes) (on_board yes) (dnp no) (fields_autoplaced)
-    (property "Reference" "R17" (at 126.4412 71.7463 90)
+    (property "Reference" "R18" (at 126.4412 71.7463 90)
       (effects (font (size 1.27 1.27)) (justify right))
     )
@@
       (project "Oro Link rev2"
         (path "/e89dcd22-1250-4a5b-b778-1c95a0dd623d/259c9346-7ad9-40c3-9e14-9b19afc78ddf"
-          (reference "R17") (unit 1)
+          (reference "R18") (unit 1)
         )
       )
