File: system-ethernet.kicad_sch (KiCad schematic)
At the start: 34 parts, among them IC9 KSZ8041RNL-TR, J6 SS-60300-103, T2 PT61017XPEL, Y1 25MHz

Commit message: first round of revisions
Parts:
- removed L?: 60R 80mA, BLM02AX100SN1D, symbol SamacSys_Parts:74279260
- added L3: BLM02PX600SN1D, BLM02AX100SN1D, symbol Oro:FerriteBead
- L?: value 60R 80mA -> BLM02PX600SN1D; symbol SamacSys_Parts:74279260 -> Oro:FerriteBead
- renumbered IC9 to IC6, R29 to R30, R30 to R31
Connections:
- net +3V3: now also L3.1
- net at C16.1, R10.2, R9.2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: now also L3.2
Other:
- moved on the sheet: R?
