File: usb-port.kicad_sch (KiCad schematic)
At the start: 5 parts, among them J7 292317-4

Commit message: first round of revisions
Parts:
- FB6: renamed from L2; symbol SamacSys_Parts:74279260 -> Oro:FerriteBead; Mouser Price/Stock (none) -> https://www.mouser.de/ProductDetail/Wurth-Elektronik/742792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
- J7: Note (none) -> USB TYPE B PORT
Changed lines of the file:
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@@
     (stroke (width 0) (type default))
   )
-  (wire (pts (xy 85.09 119.38) (xy 114.3 119.38))
+  (wire (pts (xy 90.17 119.38) (xy 114.3 119.38))
     (stroke (width 0) (type default))
   )
@@
     (stroke (width 0) (type default))
   )
-  (wire (pts (xy 85.09 114.3) (xy 86.36 114.3))
+  (wire (pts (xy 90.17 114.3) (xy 92.71 114.3))
     (stroke (width 0) (type default))
   )
@@
     (stroke (width 0) (type default))
   )
-  (wire (pts (xy 85.09 116.84) (xy 111.76 116.84))
+  (wire (pts (xy 90.17 116.84) (xy 111.76 116.84))
     (stroke (width 0) (type default))
   )
@@
     (stroke (width 0) (type default))
   )
-  (wire (pts (xy 106.68 114.3) (xy 109.22 114.3))
+  (wire (pts (xy 105.41 114.3) (xy 109.22 114.3))
     (stroke (width 0) (type default))
   )
@@
     (stroke (width 0) (type default))
   )
-  (hierarchical_label "D+" (shape bidirectional) (at 85.09 119.38 180) (fields_autoplaced)
+  (hierarchical_label "D+" (shape bidirectional) (at 90.17 119.38 180) (fields_autoplaced)
     (effects (font (size 1.27 1.27)) (justify right))
   )
-  (hierarchical_label "D-" (shape bidirectional) (at 85.09 116.84 180) (fields_autoplaced)
+  (hierarchical_label "D-" (shape bidirectional) (at 90.17 116.84 180) (fields_autoplaced)
     (effects (font (size 1.27 1.27)) (justify right))
   )
-  (hierarchical_label "VBUS" (shape input) (at 85.09 114.3 180) (fields_autoplaced)
+  (hierarchical_label "VBUS" (shape input) (at 90.17 114.3 180) (fields_autoplaced)
     (effects (font (size 1.27 1.27)) (justify right))
   )
@@
   )
   (symbol (lib_id "SamacSys_Parts:292317-4") (at 116.84 114.3 0) (unit 1)
-    (in_bom yes) (on_board yes) (dnp no) (fields_autoplaced)
+    (in_bom yes) (on_board yes) (dnp no)
     (property "Reference" "J7" (at 128.27 108.8009 0)
       (effects (font (size 1.27 1.27)))
@@
     (property "Mouser Testing Price/Stock" "" (at 135.89 139.7 0)
       (effects (font (size 1.27 1.27)) (justify left) hide)
+    )
+    (property "Note" "USB TYPE B PORT" (at 128.27 123.19 0)
+      (effects (font (size 1.27 1.27)))
     )
     (pin "1")
@@
     )
   )
-  (symbol (lib_id "SamacSys_Parts:74279260") (at 86.36 114.3 0) (unit 1)
-    (in_bom yes) (on_board yes) (dnp no) (fields_autoplaced)
-    (property "Reference" "L2" (at 96.52 110.1207 0)
-      (effects (font (size 1.27 1.27)))
-    )
-    (property "Value" "74279260" (at 96.52 112.0417 0)
-      (effects (font (size 1.27 1.27)))
-    )
-    (property "Footprint" "LEDC1608X80N" (at 102.87 113.03 0)
-      (effects (font (size 1.27 1.27)) (justify left) hide)
-    )
-    (property "Datasheet" "" (at 102.87 115.57 0)
-      (effects (font (size 1.27 1.27)) (justify left) hide)
-    )
-    (property "Description" "SMD EMI Suppression Ferrite Beads WE-CBF" (at 102.87 118.11 0)
-      (effects (font (size 1.27 1.27)) (justify left) hide)
-    )
-    (property "Height" "0.8" (at 102.87 120.65 0)
-      (effects (font (size 1.27 1.27)) (justify left) hide)
-    )
-    (property "Manufacturer_Name" "Wurth Elektronik" (at 102.87 123.19 0)
-      (effects (font (size 1.27 1.27)) (justify left) hide)
-    )
-    (property "Manufacturer_Part_Number" "74279260" (at 102.87 125.73 0)
-      (effects (font (size 1.27 1.27)) (justify left) hide)
-    )
-    (property "Mouser Part Number" "710-74279260" (at 102.87 128.27 0)
-      (effects (font (size 1.27 1.27)) (justify left) hide)
-    )
-    (property "Mouser Price/Stock" "" (at 102.87 130.81 0)
-      (effects (font (size 1.27 1.27)) (justify left) hide)
-    )
-    (property "Arrow Part Number" "" (at 102.87 133.35 0)
-      (effects (font (size 1.27 1.27)) (justify left) hide)
-    )
-    (property "Arrow Price/Stock" "" (at 102.87 135.89 0)
+  (symbol (lib_id "Oro:FerriteBead") (at 92.71 114.3 0) (unit 1)
+    (in_bom yes) (on_board yes) (dnp no)
+    (property "Reference" "FB6" (at 99.06 109.22 0)
+      (effects (font (size 1.27 1.27)))
+    )
+    (property "Value" "74279260" (at 99.06 110.49 0)
+      (effects (font (size 1.27 1.27)) (justify top))
+    )
+    (property "Footprint" "LEDC1608X80N" (at 109.22 113.03 0)
+      (effects (font (size 1.27 1.27)) (justify left) hide)
+    )
+    (property "Datasheet" "https://www.mouser.de/datasheet/2/445/74279260-3092477.pdf" (at 109.22 115.57 0)
+      (effects (font (size 1.27 1.27)) (justify left) hide)
+    )
+    (property "Description" "SMD EMI Suppression Ferrite Beads WE-CBF" (at 109.22 118.11 0)
+      (effects (font (size 1.27 1.27)) (justify left) hide)
+    )
+    (property "Height" "0.8" (at 109.22 120.65 0)
+      (effects (font (size 1.27 1.27)) (justify left) hide)
+    )
+    (property "Manufacturer_Name" "Wurth Elektronik" (at 109.22 123.19 0)
+      (effects (font (size 1.27 1.27)) (justify left) hide)
+    )
+    (property "Manufacturer_Part_Number" "74279260" (at 109.22 125.73 0)
+      (effects (font (size 1.27 1.27)) (justify left) hide)
+    )
+    (property "Mouser Part Number" "710-74279260" (at 109.22 128.27 0)
+      (effects (font (size 1.27 1.27)) (justify left) hide)
+    )
+    (property "Mouser Price/Stock" "https://www.mouser.de/ProductDetail/Wurth-Elektronik/74279260?qs=5twSNpOB8IA6LnYm%252BqxguQ%3D%3D" (at 109.22 130.81 0)
+      (effects (font (size 1.27 1.27)) (justify left) hide)
+    )
+    (property "Arrow Part Number" "" (at 109.22 133.35 0)
+      (effects (font (size 1.27 1.27)) (justify left) hide)
+    )
+    (property "Arrow Price/Stock" "" (at 109.22 135.89 0)
       (effects (font (size 1.27 1.27)) (justify left) hide)
     )
@@
       (project "Oro Link rev2"
         (path "/e89dcd22-1250-4a5b-b778-1c95a0dd623d/cb9cb53b-814d-4bdc-b9ad-369142f8d2c5"
-          (reference "L2") (unit 1)
-        )
-      )
+          (reference "FB6") (unit 1)
+        )
+      )
