File: Oro Link rev2.kicad_pcb (KiCad board)
At the start: 2 copper layers, 172 parts, among them IC1 PIC32MZ2048EFG064-E_PT, IC10 LP55231SQX_NOPB, IC2 TPS73733DCQ, IC3 PMV20ENR, IC4 PMV20ENR, IC5 PMV20ENR, IC6 TPS6734IDR, IC7 SN75C3232EPWR, IC8 ENC28J60-I_SO, IC9 KSZ8041RNL-TR, J1 42820-5223, J2 855-M50-3500542, J3 3-2328724-1, J4 5-534206-2, J5 855-M50-3500542, J6 OroConn6p, J7 292317-4, J8 SS-60300-103, J9 SS-60300-103, T1 PT61017XPEL, T2 PT61017XPEL, Y1 25MHz, Y2 25MHz

Commit message: begin refactor for rev3
Parts:
- removed C62: .47u, SamacSys_Parts:CAPC0603X33N
- removed C63: 1u, SamacSys_Parts:CAPC1608X90N
- removed IC10: LP55231SQX_NOPB, SamacSys_Parts:QFN50P400X400X80-25N
- removed L5: 60R 80mA, SamacSys_Parts:BLM02AX100SN1D
- removed the R43 at (199.8, 111.2)
- removed R46, R49: 1K, SamacSys_Parts:RESC2012X60N
- removed R47, R50: 470R, SamacSys_Parts:RESC2012X60N
- removed R48, R51: 3.3k, SamacSys_Parts:RESC1608X55N
- added FB9: BLM02PX600SN1D, SamacSys_Parts:BLM02AX100SN1D, F.Cu at (132.9, 140.7)
- added IC7: IS31FL3218-GRLS2, SamacSys_Parts:SOIC127P1036X265-24N, F.Cu at (191.1, 116.1)
- added R12: 1K, SamacSys_Parts:RESC2012X60N, F.Cu at (121.7, 112.2)
- C11, C12, C13, C37: value 10uF -> 10u
- C15: value 0.01uF -> 0.01u
- C17: value 0.047uF -> 0.047u
- C19: value 0.001uF -> 0.001u
- C20, C23: value 33uF -> 33u
- C60: value 1u -> 0.1u; footprint SamacSys_Parts:CAPC1608X90N -> SamacSys_Parts:CAPC0402X22N
- C61: value .47u -> 1u; footprint SamacSys_Parts:CAPC0603X33N -> SamacSys_Parts:CAPC1608X90N
- FB5: renamed from L1; value 18uH -> CD54NP-180MC
- FB7: renamed from L3; value 60R 80mA -> BLM02PX600SN1D
- FB8: renamed from L4; value 60R 80mA -> BLM02PX600SN1D
- LED3, LED4, LED5: value 150505M173300 -> 150120M173000; footprint SamacSys_Parts:150505M173300 -> SamacSys_Parts:150120M173000
- R44: value 470R -> 3.3k; footprint SamacSys_Parts:RESC2012X60N -> SamacSys_Parts:RESC1608X55N
- R45: value 3.3k -> 1K; footprint SamacSys_Parts:RESC1608X55N -> SamacSys_Parts:RESC2012X60N
- moved C6 146.5 mm to (96.5, 127.6)
- moved C7 146.5 mm to (96.5, 129.3)
- moved C1 140.2 mm to (96.5, 119.1)
- moved C2 140.2 mm to (96.5, 120.8)
- moved C3 140.2 mm to (96.5, 122.5)
- moved C4 140.2 mm to (96.5, 124.2)
- moved C5 140.2 mm to (96.5, 125.9)
- moved C10 138.5 mm to (98.8, 122.5)
- moved C8 138.5 mm to (98.8, 119.1)
- moved C9 138.5 mm to (98.8, 120.8)
- moved C33 126.5 mm to (98.8, 124.2)
- moved J3 124.1 mm to (102.3, 133.4)
- moved C38 122.9 mm to (98.8, 125.9)
- moved C39 122.9 mm to (98.8, 127.6)
- moved C41 122.9 mm to (98.8, 129.3)
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- renumbered L2 to FB6, IC6 to IC3, IC7 to IC4, IC8 to IC5, IC9 to IC6, IC3 to Q1, IC4 to Q2, IC5 to Q3, R12 to R13, R13 to R14, R14 to R15, R15 to R16, R16 to R17, R17 to R18, R18 to R19, R19 to R20, R20 to R21, R21 to R22, R22 to R23, R23 to R24, R24 to R25, R25 to R26, R26 to R27, R27 to R28, R28 to R29, R29 to R30, R30 to R31, R31 to R32, R32 to R33, R33 to R34, R34 to R35, R35 to R36, R36 to R37, R37 to R38, R38 to R39, R39 to R40, R40 to R41, R41 to R42, R42 to R43
Connections:
- C18 pad 2: Net-(C18-Pad2) -> /OLED Socket/EXTCAP3
- C38 pad 1: /External Ethernet/TPIN- -> Net-(C38-Pad1)
- C61 pad 1: Net-(IC10-C1+) -> GND
- C61 pad 2: Net-(IC10-C1-) -> +3V3
- D4 pad 9: unconnected-(D4-I/O_5-Pad9) -> /OLED Socket/EXTCAP3
- IC2 pad 5: +5V -> Net-(IC2-EN)
- IC6 pad 30: unconnected-(IC9-LED0_/_NWAYEN-Pad30) -> /System Ethernet/GLED+
- IC6 pad 31: unconnected-(IC9-LED1_/_SPEED-Pad31) -> /System Ethernet/YLED+
- J3 pad 5: Net-(C18-Pad2) -> /OLED Socket/EXTCAP3
- LED3 pad 1: GND -> /Indicator Lights/O15
- LED3 pad 2: Net-(LED3-A_B) -> +3V3
- LED3 pad 3: GND -> /Indicator Lights/O13
- LED3 pad 4: Net-(LED3-A_R) -> /Indicator Lights/O14
- LED4 pad 1: GND -> /Indicator Lights/O12
- LED4 pad 2: Net-(LED4-A_B) -> +3V3
- LED4 pad 3: GND -> /Indicator Lights/O10
- LED4 pad 4: Net-(LED4-A_R) -> /Indicator Lights/O11
- LED5 pad 1: GND -> /Indicator Lights/O9
- LED5 pad 2: Net-(LED5-A_B) -> +3V3
- LED5 pad 3: GND -> /Indicator Lights/O7
- LED5 pad 4: Net-(LED5-A_R) -> /Indicator Lights/O8
- R21 pad 2: /External Ethernet/TPIN- -> Net-(C38-Pad1)
- R22 pad 2: /External Ethernet/TPIN- -> Net-(C38-Pad1)
- R44 pad 1: /Indicator Lights/D2 -> GND
- R44 pad 2: Net-(LED3-A_R) -> Net-(IC7-R_EXT)
- R45 pad 1: /Indicator Lights/D3 -> Net-(IC7-~{SDB})
- R45 pad 2: Net-(LED3-A_G) -> +3V3

Commit message: fully move to new MCU configuration
Parts:
- removed C33: 0.1u, SamacSys_Parts:CAPC0402X22N
- removed C59: 1nF 5kV, SamacSys_Parts:CAPC5664X270N
- removed FB9: BLM02PX600SN1D, SamacSys_Parts:BLM02AX100SN1D
- removed R17: 10k, SamacSys_Parts:RESC5025X65N
- removed R18: 1k, SamacSys_Parts:RESC6432X65N
- removed R41: 470R, SamacSys_Parts:RESC2012X60N
- removed R42, R43: 75R, SamacSys_Parts:RESC1005X40N
- added C62: 0.1u, SamacSys_Parts:CAPC0402X22N, F.Cu at (262.5, 93.7)
- added C63: 0.1u, SamacSys_Parts:CAPC0402X22N, F.Cu at (262.5, 95.4)
- added C64: 0.1u, SamacSys_Parts:CAPC0402X22N, F.Cu at (262.5, 97.1)
- added C65: 0.1u, SamacSys_Parts:CAPC0402X22N, F.Cu at (262.5, 98.8)
- added C66: 0.1u, SamacSys_Parts:CAPC0402X22N, F.Cu at (262.5, 100.4)
- added C67: 4.7u, SamacSys_Parts:CAPC2012X135N, F.Cu at (265.6, 103.4)
- added C68: 2.2u, SamacSys_Parts:CAPC1608X90N, F.Cu at (265.4, 94.0)
- added C69: 2.2u, SamacSys_Parts:CAPC1608X90N, F.Cu at (265.4, 96.3)
- added C70: 0.1u, SamacSys_Parts:CAPC0402X22N, F.Cu at (262.5, 102.1)
- added C71: 2.2u, SamacSys_Parts:CAPC1608X90N, F.Cu at (265.4, 98.6)
- added C72: 0.1u, SamacSys_Parts:CAPC0402X22N, F.Cu at (262.5, 103.8)
- added C73: 1u, SamacSys_Parts:CAPC1608X90N, F.Cu at (265.4, 100.9)
- added C74: 0.1u, SamacSys_Parts:CAPC0402X22N, F.Cu at (262.5, 105.5)
- added IC8: STM32F479VGT6, SamacSys_Parts:QFP50P1600X1600X160-100N, F.Cu at (31.9, 7.21)
- C48: value 0.1u -> 10u; footprint SamacSys_Parts:CAPC0402X22N -> SamacSys_Parts:CAPC2012X135N
- C49: value 1u -> 0.1u; footprint SamacSys_Parts:CAPC1608X90N -> SamacSys_Parts:CAPC0402X22N
- C51, C58: value 0.1u -> 1nF 5kV; footprint SamacSys_Parts:CAPC0402X22N -> SamacSys_Parts:CAPC5664X270N
- C52, C55: value 22u -> 0.1u; footprint SamacSys_Parts:CAPC2012X95N -> SamacSys_Parts:CAPC0402X22N
- C53: value 100p -> 0.1u; footprint SamacSys_Parts:CAPC1608X90N -> SamacSys_Parts:CAPC0402X22N
- C54: value 1nF 5kV -> 0.1u; footprint SamacSys_Parts:CAPC5664X270N -> SamacSys_Parts:CAPC0402X22N
- IC6: value KSZ8041RNL-TR -> ENC28J60-I_SO; footprint SamacSys_Parts:QFN50P500X500X90-33N-D -> SamacSys_Parts:SOIC127P1030X265-28N
- J6: footprint Oro Footprints:OroConn6p -> Oro Footprints:OroConn6p_WithMounts
- R30: value 6.49k -> RC1210FR-0749R9L; footprint SamacSys_Parts:RESC2012X60N -> SamacSys_Parts:RESC3126X65N
- R31: value 4.7k -> RC1210FR-0749R9L; footprint SamacSys_Parts:RESC1005X40N -> SamacSys_Parts:RESC3126X65N
- R32, R33: value 1K -> RC1210FR-0749R9L; footprint SamacSys_Parts:RESC2012X60N -> SamacSys_Parts:RESC3126X65N
- R34: value RC1210FR-0749R9L -> 2.32k, <=1%; footprint SamacSys_Parts:RESC3126X65N -> SamacSys_Parts:ERJP06__0805_
- R35, R36, R37: value RC1210FR-0749R9L -> 75R; footprint SamacSys_Parts:RESC3126X65N -> SamacSys_Parts:RESC1005X40N
- R39: value 75R -> 470R; footprint SamacSys_Parts:RESC1005X40N -> SamacSys_Parts:RESC2012X60N
- moved IC1 193.2 mm to (31.7, 23.8)
- moved C22 179.9 mm to (48.9, 158.0)
- moved C16 179.9 mm to (48.9, 153.3)
- moved C18 179.9 mm to (48.9, 155.6)
- moved FB1 178.0 mm to (26.5, 32.3)
- moved FB2 178.0 mm to (26.5, 34.9)
- moved FB3 178.0 mm to (26.5, 37.4)
- moved FB4 178.0 mm to (26.5, 40.0)
- moved D4 177.2 mm to (33.6, 160.1)
- moved FB5 174.7 mm to (43.8, 147.2)
- moved R3 172.6 mm to (34.8, 34.3)
- moved R2 172.6 mm to (34.8, 32.1)
- moved D3 162.3 mm to (43.6, 169.0)
- moved R1 162.0 mm to (20.7, 18.7)
- moved R4 162.0 mm to (20.7, 22.9)
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Connections:
- C1 pad 2: /Microcontroller/VDD1 -> +3V3
- C2 pad 2: /Microcontroller/VDD1 -> +3V3
- C3 pad 2: /Microcontroller/VDD1 -> +3V3
- C48 pad 1: Net-(IC6-VDDPLL_1.8) -> GND
- C48 pad 2: GND -> Net-(IC6-VCAP)
- C49 pad 1: Net-(IC6-VDDPLL_1.8) -> Net-(C49-Pad1)
- C50 pad 1: +3V3 -> Net-(T2-CT_1)
- C51 pad 1: Net-(IC6-VDDA_3.3) -> GND
- C51 pad 2: GND -> Net-(C51-Pad2)
- C52 pad 1: Net-(IC6-VDDA_3.3) -> +3V3
- C53 pad 1: GND -> +3V3
- C53 pad 2: Net-(IC6-REXT) -> GND
- C54 pad 1: GND -> +3V3
- C57 pad 1: /System Ethernet/TPIN- -> +3V3
- C58 pad 1: Net-(T2-CT_1) -> GND
- C6 pad 2: /Microcontroller/VDD2 -> +3V3
- C7 pad 2: /Microcontroller/VDD2 -> +3V3
- C8 pad 2: /Microcontroller/VDD2 -> +3V3
- D6 pad 1: /Microcontroller/SERIAL_TX -> /UART Port/TX
- D6 pad 2: /Microcontroller/SERIAL_RX -> /UART Port/RX
- D6 pad 4: /Microcontroller/SERIAL_RTS -> /UART Port/RTS
- D6 pad 5: /Microcontroller/SERIAL_CTS -> /UART Port/CTS
- D8 pad 1: /ISCP Pad/PGEC -> /JTAG Pad/PGEC
- D8 pad 2: /ISCP Pad/PGED -> /JTAG Pad/PGED
- D8 pad 5: /ISCP Pad/~{MCLR} -> /JTAG Pad/~{MCLR}
- D9 pad 2: /Microcontroller/USB_D- -> /USB Port/D-
- D9 pad 4: /Microcontroller/USB_D+ -> /USB Port/D+
- FB2 pad 2: /Microcontroller/VDD1 -> +3V3
- FB4 pad 2: /Microcontroller/VDD2 -> +3V3
- FB6 pad 1: +5V -> /USB Port/VBUS
- FB8 pad 2: Net-(IC6-VDDA_3.3) -> Net-(T2-CT_1)
- IC1 pad 10: /External Ethernet/~{RST} -> /Microcontroller/EXTETH_~{RST}
- IC1 pad 12: /Front Panel Client/PWR_ON -> /Microcontroller/FP_PWR
- IC1 pad 13: /Front Panel Client/RESET -> /Microcontroller/FP_RST
- IC1 pad 14: /Power Supply/PW_ON -> /Microcontroller/PSU_PSON
- IC1 pad 15: /ISCP Pad/PGEC -> /Microcontroller/ICSP_PGEC
- IC1 pad 16: /ISCP Pad/PGED -> /Microcontroller/ICSP_PGED
- IC1 pad 26: /Microcontroller/VDD2 -> +3V3
- IC1 pad 29: /External Ethernet/SCK -> /Microcontroller/EXTETH_SCK
- IC1 pad 32: /OLED Socket/~{RST} -> /Microcontroller/OLED_~{RST}
- IC1 pad 34: /Microcontroller/VDD2 -> +3V3
- IC1 pad 38: /Power Supply/PW_OK -> /Microcontroller/PSU_PSOK
- IC1 pad 39: /Microcontroller/VDD2 -> +3V3
- IC1 pad 4: /External Ethernet/~{CS} -> /Microcontroller/EXTETH_~{CS}
- IC1 pad 41: /COM Bus Header/RTS -> /Microcontroller/SYSSERIAL_RTS
- IC1 pad 42: /COM Bus Header/CTS -> /Microcontroller/SYSSERIAL_CTS
- IC1 pad 43: /COM Bus Header/TX -> /Microcontroller/SYSSERIAL_TX
- IC1 pad 44: /OLED Socket/SCK -> /Microcontroller/OLED_SCK
- IC1 pad 45: /OLED Socket/SDI -> /Microcontroller/OLED_SDO
- IC1 pad 46: /COM Bus Header/RX -> /Microcontroller/SYSSERIAL_RX
- IC1 pad 47: /External Ethernet/SDI -> /Microcontroller/EXTETH_SDO
- IC1 pad 48: /External Ethernet/SDO -> /Microcontroller/EXTETH_SDI
- IC1 pad 5: /Indicator Lights/SDA -> /Microcontroller/I2C_SDA
- IC1 pad 52: /External Ethernet/~{INT} -> /Microcontroller/EXTETH_INT
- IC1 pad 54: /Microcontroller/VDD1 -> +3V3
- IC1 pad 6: /Indicator Lights/SCL -> /Microcontroller/I2C_SCL
- IC1 pad 60: /Microcontroller/VDD1 -> +3V3
- IC1 pad 8: /Microcontroller/VDD1 -> +3V3
- IC1 pad 9: /ISCP Pad/~{MCLR} -> /Microcontroller/ISCP_~{MCLR}
- IC6 pad 1: GND -> Net-(IC6-VCAP)
- IC6 pad 10: Net-(IC6-REXT) -> /System Ethernet/~{RST}
- IC6 pad 11: /Microcontroller/ETH_MDIO -> GND
- IC6 pad 12: /Microcontroller/ETH_EMDC -> /System Ethernet/TPIN-
- IC6 pad 13: Net-(IC6-PHYAD0) -> /System Ethernet/TPIN+
- IC6 pad 14: Net-(IC6-PHYAD0) -> Net-(IC6-RBIAS)
- IC6 pad 15: /Microcontroller/ETH_ERXD1 -> +3V3
- IC6 pad 16: /Microcontroller/ETH_ERXD0 -> /System Ethernet/TPOUT-
- IC6 pad 17: +3V3 -> /System Ethernet/TPOUT+
- IC6 pad 18: /Microcontroller/ETH_ECRSDV -> GND
- IC6 pad 19: /Microcontroller/ETH_EREFCLK -> +3V3
- IC6 pad 2: Net-(IC6-VDDPLL_1.8) -> GND
- IC6 pad 20: /Microcontroller/ETH_ERXERR -> +3V3
- IC6 pad 21: /Microcontroller/ETH_INT -> GND
- IC6 pad 22: unconnected-(IC6-NC_1-Pad22) -> GND
- IC6 pad 23: /Microcontroller/ETH_ETXEN -> Net-(IC6-OSC1)
- IC6 pad 24: /Microcontroller/ETH_ETXD0 -> unconnected-(IC6-OSC2-Pad24)
- IC6 pad 25: /Microcontroller/ETH_ETXD1 -> +3V3
- IC6 pad 26: unconnected-(IC6-NC_2-Pad26) -> /System Ethernet/YLED+
- IC6 pad 27: unconnected-(IC6-NC_3-Pad27) -> /System Ethernet/GLED+
- IC6 pad 28: Net-(IC6-CONFIG0) -> +3V3
- IC6 pad 3: Net-(IC6-VDDA_3.3) -> unconnected-(IC6-CLKOUT-Pad3)
- IC6 pad 4: /System Ethernet/TPIN- -> /System Ethernet/~{INT}
- IC6 pad 5: /System Ethernet/TPIN+ -> unconnected-(IC6-NC-Pad5)
- IC6 pad 6: /System Ethernet/TPOUT- -> /System Ethernet/SDO
- IC6 pad 7: /System Ethernet/TPOUT+ -> /System Ethernet/SDI
- IC6 pad 8: unconnected-(IC6-XO-Pad8) -> /System Ethernet/SCK
- IC6 pad 9: Net-(IC6-XI) -> /System Ethernet/~{CS}
- J4 pad 1: /Microcontroller/SERIAL_TX -> /UART Port/TX
- J4 pad 2: /Microcontroller/SERIAL_RX -> /UART Port/RX
- J4 pad 3: /Microcontroller/SERIAL_RTS -> /UART Port/RTS
- J4 pad 4: /Microcontroller/SERIAL_CTS -> /UART Port/CTS
- J6 pad 3: /ISCP Pad/PGED -> /JTAG Pad/PGED
- J6 pad 4: /ISCP Pad/PGEC -> /JTAG Pad/PGEC
- J6 pad 5: /ISCP Pad/~{MCLR} -> /JTAG Pad/~{MCLR}
- J7 pad 2: /Microcontroller/USB_D- -> /USB Port/D-
- J7 pad 3: /Microcontroller/USB_D+ -> /USB Port/D+
- R2 pad 2: /Indicator Lights/SDA -> /Microcontroller/I2C_SDA
- R3 pad 2: /Indicator Lights/SCL -> /Microcontroller/I2C_SCL
- R30 pad 1: GND -> /System Ethernet/TPOUT+
- R30 pad 2: Net-(IC6-REXT) -> Net-(T2-CT_1)
- R31 pad 1: +3V3 -> /System Ethernet/TPOUT-
- R31 pad 2: /Microcontroller/ETH_MDIO -> Net-(T2-CT_1)
- R32 pad 1: Net-(IC6-PHYAD0) -> /System Ethernet/TPIN+
- R32 pad 2: GND -> Net-(C49-Pad1)
- R33 pad 1: Net-(IC6-CONFIG0) -> /System Ethernet/TPIN-
- R33 pad 2: +3V3 -> Net-(C49-Pad1)
- R34 pad 1: /System Ethernet/TPOUT+ -> Net-(IC6-RBIAS)
- R34 pad 2: Net-(T2-CT_1) -> GND
- R35 pad 1: /System Ethernet/TPOUT- -> Net-(T2-CT_3)
- R35 pad 2: Net-(T2-CT_1) -> Net-(C51-Pad2)
- R36 pad 1: /System Ethernet/TPIN+ -> Net-(T2-CT_4)
- R36 pad 2: /System Ethernet/TPIN- -> Net-(C51-Pad2)
- R37 pad 1: /System Ethernet/TPIN- -> /System Ethernet/CT_45
- R37 pad 2: /System Ethernet/TPIN- -> Net-(C51-Pad2)
- R38 pad 1: Net-(T2-CT_3) -> /System Ethernet/CT_78
- R38 pad 2: Net-(C59-Pad2) -> Net-(C51-Pad2)
- R39 pad 1: Net-(T2-CT_4) -> Net-(J9-ANODE_GREEN/CATHODE_YELLOW_1)
- R39 pad 2: Net-(C59-Pad2) -> /System Ethernet/GLED+
- R40 pad 1: Net-(J9-ANODE_GREEN/CATHODE_YELLOW_1) -> Net-(J9-ANODE_YELLOW/CATHODE_GREEN_2)
- R40 pad 2: /System Ethernet/GLED+ -> /System Ethernet/YLED+
- Y2 pad 3: Net-(IC6-XI) -> Net-(IC6-OSC1)
Other:
- board outline added: 40.1 x 35.6 mm

Commit message: first few boards laid out
Parts:
- removed the C10 at (31.9, 38.7)
- removed the C2 at (29.6, 33.6)
- removed the C25 at (43.3, 156.1)
- removed the C3 at (29.6, 35.3)
- removed the C35 at (146.1, 82.7)
- removed the C36 at (153.7, 82.7)
- removed the C4 at (29.6, 37.0)
- removed the C5 at (29.6, 38.7)
- removed the C6 at (31.9, 31.9)
- removed the C7 at (31.9, 33.6)
- removed the C8 at (31.9, 35.3)
- removed the C9 at (31.9, 37.0)
- removed the D4 at (33.6, 160.1)
- removed the D5 at (33.5, 168.0)
- removed the FB1 at (26.5, 32.3)
- removed the FB2 at (26.5, 34.9)
- removed the FB3 at (26.5, 37.4)
- removed FB4: BMC1JY0300AN, SamacSys_Parts:BEADC1608X95N
- removed FB6: 74279260, SamacSys_Parts:LEDC1608X80N
- removed the IC1 at (31.7, 23.8)
- removed the R1 at (20.7, 18.7)
- removed the R11 at (20.7, 52.7)
- removed the R13 at (77.8, 62.2)
- removed the R14 at (140.0, 33.4)
- removed the R15 at (140.0, 36.3)
- removed R45: 1K, SamacSys_Parts:RESC2012X60N
- added C18: 1nF 5kV, SamacSys_Parts:CAPC5664X270N, F.Cu at (472.3, -129.2)
- added CR1: BYV10D-600PJ, BYV10D-600PJ:BYV10D-600PJ, F.Cu at (457.3, 275.9)
- added J10: 690367180872, SamacSys_Parts:690367180872, F.Cu at (94.6, 106.6)
- added J11: 690367180872, SamacSys_Parts:690367180872, F.Cu at (139.8, 96.2)
- added J12: 690367180872, SamacSys_Parts:690367180872, F.Cu at (130.4, 125.1)
- added J13: 690367180872, SamacSys_Parts:690367180872, F.Cu at (128.1, 82.7)
- added J14: 690357100872, Oro Footprints:690357100872, B.Cu at (525.1, -132.5)
- added J15: 690357100872, Oro Footprints:690357100872, B.Cu at (478.4, 81.1)
- added J16: 690357100872, Oro Footprints:690357100872, B.Cu at (479.4, 267.5)
- added J17: 690357100872, Oro Footprints:690357100872, B.Cu at (476.7, -35.8)
- added J18: 690357100872, Oro Footprints:690357100872, B.Cu at (278.5, 60.2)
- added J19: 42820-5214, SamacSys_Parts:42820-5XXY_1, F.Cu at (518.5, -158.4)
- added J2: 690357100872, Oro Footprints:690357100872, B.Cu at (-260.2, 5.12)
- added J25: 10129378-902003BLF, SamacSys_Parts:HDRV2W67P0X254_1X2_508X241X1082P, F.Cu at (-256.1, -156.7)
- added J26: 10129378-902003BLF, SamacSys_Parts:HDRV2W67P0X254_1X2_508X241X1082P, F.Cu at (-256.1, -152.5)
- added J3: 690357100872, Oro Footprints:690357100872, B.Cu at (-255.8, -71.0)
- added J5: 690367180872, SamacSys_Parts:690367180872, F.Cu at (139.8, 113.3)
- added J6: 690367180872, SamacSys_Parts:690367180872, F.Cu at (95.9, 125.1)
- added J8: 690367180872, SamacSys_Parts:690367180872, F.Cu at (111.4, 82.7)
- added J9: 690367180872, SamacSys_Parts:690367180872, F.Cu at (113.1, 125.1)
- added LED1: AA3528VRVFS/A, SamacSys_Parts:AA3528VRVFSA, F.Cu at (119.8, 117.5)
- added R24: 10k, SamacSys_Parts:RESC5025X65N, F.Cu at (-264.8, -63.3)
- added R3: 10k, SamacSys_Parts:RESC5025X65N, F.Cu at (111.3, 91.6)
- added R37: 10k, SamacSys_Parts:RESC5025X65N, F.Cu at (261.7, 63.6)
- added S1: TL6400AF160QJ, SamacSys_Parts:TL6400AF160QJ, F.Cu at (106.4, 111.7)
- added X1: 7P-26.000MBP-T, Oro Footprints:7P-26.000MBP-T, F.Cu at (109.0, 97.1)
- added mouse-bite-2.54mm-slot: VAL**, panelization:mouse-bite-2.54mm-slot, F.Cu at (104.2, 79.2)
- C26: renamed from C17; footprint SamacSys_Parts:C1608_Commercial -> Oro Footprints:C1608_Commercial_Tight
- C27: renamed from C19; footprint SamacSys_Parts:C1608_Commercial -> Oro Footprints:C1608_Commercial_Tight
- D9: value PESD4USB5B-TBSX -> P6SMB15A-Q; footprint SamacSys_Parts:PESD4USB5BTBSX -> SamacSys_Parts:DIOM5436X244N
- FB2: renamed from FB8; value BLM02PX600SN1D -> BLM18BB600SZ1D; footprint SamacSys_Parts:BLM02AX100SN1D -> SamacSys_Parts:BLM18EG121SH1D
- FB3: renamed from FB7; value BLM02PX600SN1D -> BLM18BB600SZ1D; footprint SamacSys_Parts:BLM02AX100SN1D -> SamacSys_Parts:BLM18EG121SH1D
- J1: value 42820-5223 -> 690357100872; footprint SamacSys_Parts:42820-5XXY_1 -> Oro Footprints:690357100872; moved to B.Cu
- J4: value 5-534206-2 -> 690357100872; footprint SamacSys_Parts:RHDR4W77P254_2X2_508X503X864P -> Oro Footprints:690357100872; moved to B.Cu
- J7: value 292317-4 -> 690367180872; footprint SamacSys_Parts:2923174 -> SamacSys_Parts:690367180872
- LED3: renamed from LED2; value AA3528VRVFS/A -> CLM3C-WKW-CXAYA453
- R12: value 1K -> 10k; footprint SamacSys_Parts:RESC2012X60N -> SamacSys_Parts:RESC5025X65N
- R4, R6, R7: value 10k -> 1k; footprint SamacSys_Parts:RESC5025X65N -> SamacSys_Parts:RESC2012X60N
- moved R5 522.1 mm to (521.6, -120.1)
- moved D4 518.8 mm to (-249.7, 13.3)
- moved J22 513.1 mm to (-265.0, -16.1)
- moved R18 513.1 mm to (-242.0, -2.53)
- moved R19 513.1 mm to (-242.0, -0.38)
- moved R20 513.1 mm to (-242.0, 1.77)
- moved R21 513.1 mm to (-242.0, 3.92)
- moved C31 513.1 mm to (-244.8, -2.76)
- moved C32 513.1 mm to (-244.8, -1.07)
- moved C33 513.1 mm to (-269.1, 0.38)
- moved C34 513.1 mm to (-244.8, 0.62)
- moved C35 513.1 mm to (-244.8, 2.31)
- moved C36 513.1 mm to (-244.8, 4.00)
- moved C37 513.1 mm to (-244.8, 5.69)
- moved C38 513.1 mm to (-244.8, 7.38)
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- renumbered C70 to C10, C74 to C11, C71 to C12, C72 to C13, C73 to C14, C11 to C15, C12 to C16, C13 to C17, C14 to C19, C67 to C2, C16 to C20, C18 to C21, C21 to C22, C22 to C23, C15 to C25, C20 to C28, C23 to C29, C68 to C3, C48 to C30, C49 to C31, C50 to C32, C51 to C33, C52 to C34, C53 to C35, C54 to C36, C55 to C37, C56 to C38, C57 to C39, C69 to C4, C58 to C40, C37 to C41, C38 to C42, C39 to C43, C40 to C44, C41 to C45, C42 to C46, C43 to C47, C44 to C48, C45 to C49, C62 to C5, C46 to C50, C47 to C51, C34 to C52, C26 to C53, C27 to C54, C28 to C55, C29 to C56, C30 to C57, C31 to C58, C32 to C59, C63 to C6, C64 to C7, C65 to C8, C66 to C9, D6 to D10, D7 to D11, D12 to D4, D13 to D5, D10 to D6, D11 to D7, FB5 to FB1, IC8 to IC1, IC6 to IC4, IC4 to IC6, J2 to J20, J3 to J21, J9 to J22, J8 to J23, J6 to J24, J5 to J27, LED1 to LED2, LED3 to LED4, LED4 to LED5, LED5 to LED6, R3 to R1, R16 to R11, R30 to R13, R31 to R14, R32 to R15, R33 to R16, R34 to R17, R35 to R18, R36 to R19, R37 to R20, R38 to R21, R39 to R22, R40 to R23, R19 to R25, R20 to R26, R21 to R27, R22 to R28, R23 to R29, R24 to R30, R25 to R31, R26 to R32, R27 to R33, R28 to R34, R29 to R35, R44 to R36, S1 to S2, S2 to S3, S3 to S4, T2 to T1, T1 to T2, Y2 to Y1, Y1 to Y2
Connections:
- C1 pad 1: GND -> Net-(IC1-NRST)
- C1 pad 2: +3V3 -> GND
- C19 pad 1: GND -> GNDPWR
- C33 pad 1: GND -> GNDPWR
- C40 pad 1: GND -> GNDPWR
- C44 pad 1: GND -> GNDPWR
- C51 pad 1: GND -> GNDPWR
- C52 pad 1: GND -> GNDPWR
- C53 pad 1: GND -> GNDPWR
- C59 pad 1: GND -> GNDPWR
- D1 pad 2: GND -> GNDPWR
- D10 pad 1: /UART Port/TX -> /USB+UART Ports/UART_RX
- D10 pad 2: /UART Port/RX -> /USB+UART Ports/UART_TX
- D10 pad 3: GND -> GNDPWR
- D10 pad 4: /UART Port/RTS -> /USB+UART Ports/USB_D+
- D10 pad 5: /UART Port/CTS -> /USB+UART Ports/USB_D-
- D10 pad 8: GND -> GNDPWR
- D11 pad 1: GND -> GNDPWR
- D11 pad 14: GND -> GNDPWR
- D11 pad 7: GND -> GNDPWR
- D11 pad 8: GND -> GNDPWR
- D2 pad 1: GND -> GNDPWR
- D2 pad 14: GND -> GNDPWR
- D2 pad 7: GND -> GNDPWR
- D2 pad 8: GND -> GNDPWR
- D4 pad 3: GND -> GNDPWR
- D5 pad 3: GND -> GNDPWR
- D5 pad 8: GND -> GNDPWR
- D6 pad 3: GND -> GNDPWR
- D7 pad 3: GND -> GNDPWR
- D7 pad 8: GND -> GNDPWR
- D8 pad 1: /JTAG Pad/PGEC -> /SWD Pad/SWDIO
- D8 pad 2: /JTAG Pad/PGED -> /SWD Pad/SWCLK
- D8 pad 3: GND -> GNDPWR
- D8 pad 4: +3V3 -> /SWD Pad/SWO
- D8 pad 5: /JTAG Pad/~{MCLR} -> /SWD Pad/FLASH
- D8 pad 8: GND -> GNDPWR
- D9 pad 1: Net-(D9-CH1) -> /SWD Pad/VCC
- D9 pad 2: /USB Port/D- -> GNDPWR
- H1 pad 1: GND -> GNDPWR
- H2 pad 1: GND -> GNDPWR
- H3 pad 1: GND -> GNDPWR
- H4 pad 1: GND -> GNDPWR
- H5 pad 1: GND -> GNDPWR
- IC1 pad 11: unconnected-(IC8-NRST-Pad11) -> Net-(IC1-NRST)
- IC1 pad 14: unconnected-(IC8-PC2-Pad14) -> /Microcontroller/EXTETH_MISO
- IC1 pad 15: unconnected-(IC8-PC3-Pad15) -> /Microcontroller/EXTETH_MOSI
- IC1 pad 20: unconnected-(IC8-PA1-Pad20) -> /Microcontroller/SYSUART_RTS
- IC1 pad 21: unconnected-(IC8-PA2-Pad21) -> /Microcontroller/SYSUART_TX
- IC1 pad 22: unconnected-(IC8-PA3-Pad22) -> /Microcontroller/SYSUART_RX
- IC1 pad 26: unconnected-(IC8-PA5-Pad26) -> /Microcontroller/SYSETH_SCK
- IC1 pad 27: unconnected-(IC8-PA6-Pad27) -> /Microcontroller/SYSETH_MISO
- IC1 pad 28: unconnected-(IC8-PA7-Pad28) -> /Microcontroller/SYSTEH_MOSI
- IC1 pad 29: unconnected-(IC8-PB0-Pad29) -> /Microcontroller/SYSTEH_~{RST}
- IC1 pad 30: unconnected-(IC8-PB1-Pad30) -> /Microcontroller/SYSTEH_~{INT}
- IC1 pad 32: unconnected-(IC8-PE7-Pad32) -> /Microcontroller/DBGUART_RX
- IC1 pad 33: unconnected-(IC8-PE8-Pad33) -> /Microcontroller/DBGUART_TX
- IC1 pad 37: unconnected-(IC8-PE12-Pad37) -> Net-(IC1-PE12)
- IC1 pad 4: /Microcontroller/ETH_~{RST} -> /Microcontroller/EXTETH_~{RST}
- IC1 pad 41: unconnected-(IC8-PB10-Pad41) -> /Microcontroller/EXTETH_SCK
- IC1 pad 47: unconnected-(IC8-PB13-Pad47) -> /Microcontroller/PSU_ON
- IC1 pad 48: unconnected-(IC8-PB14-Pad48) -> /Microcontroller/PSU_OK
- IC1 pad 49: unconnected-(IC8-PB15-Pad49) -> /Microcontroller/SYS_RESET
- IC1 pad 50: unconnected-(IC8-PD8-Pad50) -> /Microcontroller/SYS_POWER
- IC1 pad 73: unconnected-(IC8-PA11-Pad73) -> /Microcontroller/USB_D-
- IC1 pad 74: unconnected-(IC8-PA12-Pad74) -> /Microcontroller/USB_D+
- IC1 pad 75: unconnected-(IC8-PA13-Pad75) -> /Microcontroller/SWDIO
- IC1 pad 79: unconnected-(IC8-PA14-Pad79) -> /Microcontroller/SWCLK
- IC1 pad 81: unconnected-(IC8-PC10-Pad81) -> /Microcontroller/OLED_SCK
- IC1 pad 87: unconnected-(IC8-PD3-Pad87) -> /Microcontroller/SYSUART_CTS
- IC1 pad 89: unconnected-(IC8-PD5-Pad89) -> /Microcontroller/OLED_~{RST}
- IC1 pad 9: unconnected-(IC8-PH0-Pad9) -> Net-(IC1-PH0)
- IC1 pad 90: unconnected-(IC8-PD6-Pad90) -> /Microcontroller/OLED_MOSI
- IC1 pad 92: unconnected-(IC8-PB3-Pad92) -> /Microcontroller/SWO
- IC1 pad 95: unconnected-(IC8-PB6-Pad95) -> /Microcontroller/I2C_SCL
- IC1 pad 96: unconnected-(IC8-PB7-Pad96) -> /Microcontroller/I2C_SDA
- IC1 pad 97: unconnected-(IC8-BOOT0-Pad97) -> /Microcontroller/~{FLASH}
- IC1 pad 99: unconnected-(IC8-PB9-Pad99) -> /Microcontroller/EXTETH_~{INT}
- IC4 pad 9: /System Ethernet/~{CS} -> Net-(IC4-~{CS})
- IC5 pad 9: /External Ethernet/~{CS} -> Net-(IC5-~{CS})
- J1 pad 1: /Power Supply/5VSB -> +3V3
- J1 pad 2: /Power Supply/5VSB -> /USB+UART Ports/UART_TX
- J1 pad 3: /Power Supply/PW_OK -> /USB+UART Ports/UART_RX
- J1 pad 4: /Power Supply/PW_OK -> /USB+UART Ports/USB_D-
- J1 pad 5: /Power Supply/PSU_ON -> /USB+UART Ports/USB_D+
- J1 pad 6: /Power Supply/PSU_ON -> GND
- J1 pad 7: +5V -> GND
- J1 pad 8: +5V -> GND
- J21 pad 13: +3V3 -> Net-(J21-Pad13)
- J21 pad 14: GND -> Net-(J21-Pad14)
- J21 pad 16: GND -> Net-(J21-Pad14)
- J21 pad 17: GND -> Net-(J21-Pad17)
- J21 pad 19: GND -> Net-(J21-Pad17)
- J21 pad 20: GND -> Net-(J21-Pad14)
- J21 pad 21: GND -> Net-(J21-Pad17)
- J21 pad 24: GND -> Net-(J21-Pad14)
- J21 pad 25: GND -> Net-(J21-Pad17)
- J21 pad 26: GND -> Net-(J21-Pad14)
- J21 pad 27: GND -> Net-(J21-Pad17)
- J21 pad 28: GND -> Net-(J21-Pad14)
- J21 pad 29: GND -> Net-(J21-Pad17)
- J21 pad MP1: GND -> unconnected-(J21-PadMP1)
- J21 pad MP2: GND -> unconnected-(J21-PadMP2)
- J22 pad MH1: GND -> GNDPWR
- J22 pad MH2: GND -> GNDPWR
- J23 pad MH1: GND -> GNDPWR
- J23 pad MH2: GND -> GNDPWR
- J24 pad 1: +3V3 -> /SWD Pad/VCC
- J24 pad 3: /JTAG Pad/PGED -> /SWD Pad/FLASH
- J24 pad 4: /JTAG Pad/PGEC -> /SWD Pad/SWO
- J24 pad 5: /JTAG Pad/~{MCLR} -> /SWD Pad/SWCLK
- J24 pad 6: unconnected-(J6-Pad6) -> /SWD Pad/SWDIO
- J4 pad 1: /UART Port/TX -> +3V3
- J4 pad 2: /UART Port/RX -> +5V
- J4 pad 3: /UART Port/RTS -> /OLED Socket/~{RST}
- J4 pad 4: /UART Port/CTS -> /OLED Socket/SCK
- J7 pad 1: Net-(D9-CH1) -> +3V3
- J7 pad 2: /USB Port/D- -> /Microcontroller/EXTETH_SCK
- J7 pad 3: /USB Port/D+ -> /Microcontroller/EXTETH_MISO
- J7 pad 4: GND -> /Microcontroller/EXTETH_MOSI
- LED2 pad 2: Net-(LED1-Pad2) -> Net-(LED2-Pad2)
- LED3 pad 1: Net-(LED2-Pad1) -> Net-(LED3-Pad1)
- R10 pad 1: Net-(IC1-OSC1/CLKI/RC12) -> GND
- R10 pad 2: GND -> Net-(J21-Pad14)
- R12 pad 1: Net-(IC2-EN) -> GND
- R12 pad 2: +5V -> Net-(IC4-~{CS})
- R4 pad 1: Net-(IC1-AN48/RPB8/PMA10/RB8) -> Net-(IC1-PE12)
- R4 pad 2: GND -> Net-(LED1-Pad1)
- R5 pad 1: Net-(IC1-AN49/RPB9/PMA7/RB9) -> +5V
- R5 pad 2: GND -> Net-(IC2-EN)
- R6 pad 1: Net-(IC1-TMS/CVREFOUT/AN5/RPB10/PMA13/RB10) -> Net-(LED2-Pad2)
- R6 pad 2: GND -> /Front Panel Client/PLED+
- R7 pad 1: Net-(IC1-TDO/AN6/PMA12/RB11) -> /Front Panel Client/HDD+
- R7 pad 2: GND -> Net-(LED3-Pad1)
- R8 pad 1: Net-(IC1-TCK/AN7/PMA11/RB12) -> GND
- R8 pad 2: GND -> Net-(J21-Pad17)
- R9 pad 1: Net-(IC1-TDI/AN8/RB13) -> Net-(J21-Pad13)
- R9 pad 2: GND -> +3V3
- S2 pad MH1: GND -> GNDPWR
- S2 pad MH2: GND -> GNDPWR
Routing:
- net +5V: track 0.00 -> 85.2 mm
- net +3V3: track 0.00 -> 60.6 mm, vias 0 -> 14
- net GND: track 0.00 -> 53.7 mm, vias 0 -> 23
- net /OLED Socket/+12V: track 0.00 -> 51.4 mm
- net /Microcontroller/EXTETH_SCK: track 0.00 -> 41.7 mm, vias 0 -> 1
- net /Microcontroller/SYSUART_CTS: track 0.00 -> 39.2 mm, vias 0 -> 1
- net /OLED Socket/SDI: track 0.00 -> 38.7 mm, vias 0 -> 1
- net /OLED Socket/~{RST}: track 0.00 -> 37.4 mm, vias 0 -> 1
- net /Microcontroller/EXTETH_MISO: track 0.00 -> 35.9 mm, vias 0 -> 1
- net /Microcontroller/EXTETH_~{INT}: track 0.00 -> 35.0 mm, vias 0 -> 2
- net /OLED Socket/SCK: track 0.00 -> 33.9 mm, vias 0 -> 1
- net /Microcontroller/~{FLASH}: track 0.00 -> 31.5 mm
- net /Microcontroller/EXTETH_~{RST}: track 0.00 -> 27.4 mm, vias 0 -> 2
- net /Microcontroller/SWO: track 0.00 -> 26.5 mm
- net /Microcontroller/DBGUART_RX: track 0.00 -> 26.2 mm
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- added copper zone on In2.Cu, net +3V3
- added copper zone on B.Cu, net GND
- added copper zone on F.Cu, net GND
- added copper zone on In1.Cu, net GND
Other:
- board size 40.1 x 35.6 mm -> 25.9 x 115.8 mm
- copper layers 2 -> 4
- board text added: "OLED"
