File: com-bus-header.kicad_sch (KiCad schematic)
At the start: 11 parts, among them IC7 SN75C3232EPWR, J2 855-M50-3500542

Commit message: first round of revisions
Parts:
- renumbered IC7 to IC4
Changed lines of the file:
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@@
   (symbol (lib_id "SamacSys_Parts:SN75C3232EPWR") (at 71.12 74.93 0) (unit 1)
     (in_bom yes) (on_board yes) (dnp no)
-    (property "Reference" "IC7" (at 86.36 68.58 0)
+    (property "Reference" "IC4" (at 86.36 68.58 0)
       (effects (font (size 1.27 1.27)))
     )
@@
       (project "Oro Link rev2"
         (path "/e89dcd22-1250-4a5b-b778-1c95a0dd623d/a5104146-06a0-496e-bda0-1e4731a261c3"
-          (reference "IC7") (unit 1)
+          (reference "IC4") (unit 1)
         )
       )

Commit message: fully move to new MCU configuration
Parts:
- renumbered C27 to C55, C28 to C56, C29 to C57, C30 to C58, C31 to C59, IC4 to IC6
Changed lines of the file:
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@@
   (symbol (lib_id "SamacSys_Parts:UUP1H0R1MCL1GS") (at 92.71 125.73 180) (unit 1)
     (in_bom yes) (on_board yes) (dnp no)
-    (property "Reference" "C31" (at 91.44 127 0)
+    (property "Reference" "C59" (at 91.44 127 0)
       (effects (font (size 1.27 1.27)))
     )
@@
       (project "Oro Link rev2"
         (path "/e89dcd22-1250-4a5b-b778-1c95a0dd623d/a5104146-06a0-496e-bda0-1e4731a261c3"
-          (reference "C31") (unit 1)
+          (reference "C59") (unit 1)
         )
       )
@@
   (symbol (lib_id "SamacSys_Parts:SN75C3232EPWR") (at 71.12 74.93 0) (unit 1)
     (in_bom yes) (on_board yes) (dnp no)
-    (property "Reference" "IC4" (at 86.36 68.58 0)
+    (property "Reference" "IC6" (at 86.36 68.58 0)
       (effects (font (size 1.27 1.27)))
     )
@@
       (project "Oro Link rev2"
         (path "/e89dcd22-1250-4a5b-b778-1c95a0dd623d/a5104146-06a0-496e-bda0-1e4731a261c3"
-          (reference "IC4") (unit 1)
+          (reference "IC6") (unit 1)
         )
       )
@@
   (symbol (lib_id "power:GND") (at 165.1 97.79 0) (unit 1)
     (in_bom yes) (on_board yes) (dnp no) (fields_autoplaced)
-    (property "Reference" "#PWR065" (at 165.1 104.14 0)
+    (property "Reference" "#PWR0110" (at 165.1 104.14 0)
       (effects (font (size 1.27 1.27)) hide)
     )
@@
       (project "Oro Link rev2"
         (path "/e89dcd22-1250-4a5b-b778-1c95a0dd623d/a5104146-06a0-496e-bda0-1e4731a261c3"
-          (reference "#PWR065") (unit 1)
+          (reference "#PWR0110") (unit 1)
         )
       )
@@
         )
         (path "/e89dcd22-1250-4a5b-b778-1c95a0dd623d/a5104146-06a0-496e-bda0-1e4731a261c3"
-          (reference "C32") (unit 1)
+          (reference "C60") (unit 1)
         )
       )
@@
   (symbol (lib_id "power:GND") (at 113.03 73.66 0) (unit 1)
     (in_bom yes) (on_board yes) (dnp no) (fields_autoplaced)
-    (property "Reference" "#PWR064" (at 113.03 80.01 0)
+    (property "Reference" "#PWR0109" (at 113.03 80.01 0)
       (effects (font (size 1.27 1.27)) hide)
     )
@@
       (project "Oro Link rev2"
         (path "/e89dcd22-1250-4a5b-b778-1c95a0dd623d/a5104146-06a0-496e-bda0-1e4731a261c3"
-          (reference "#PWR064") (unit 1)
+          (reference "#PWR0109") (unit 1)
         )
       )
@@
   (symbol (lib_id "SamacSys_Parts:UUP1H0R1MCL1GS") (at 80.01 138.43 0) (unit 1)
     (in_bom yes) (on_board yes) (dnp no)
-    (property "Reference" "C30" (at 91.44 139.7 0)
+    (property "Reference" "C58" (at 91.44 139.7 0)
       (effects (font (size 1.27 1.27)))
     )
@@
       (project "Oro Link rev2"
         (path "/e89dcd22-1250-4a5b-b778-1c95a0dd623d/a5104146-06a0-496e-bda0-1e4731a261c3"
-          (reference "C30") (unit 1)
+          (reference "C58") (unit 1)
         )
       )
@@
         )
         (path "/e89dcd22-1250-4a5b-b778-1c95a0dd623d/a5104146-06a0-496e-bda0-1e4731a261c3"
-          (reference "#PWR067") (unit 1)
+          (reference "#PWR0112") (unit 1)
         )
       )
@@
   (symbol (lib_id "power:GND") (at 100.33 143.51 0) (unit 1)
     (in_bom yes) (on_board yes) (dnp no) (fields_autoplaced)
-    (property "Reference" "#PWR062" (at 100.33 149.86 0)
+    (property "Reference" "#PWR0107" (at 100.33 149.86 0)
       (effects (font (size 1.27 1.27)) hide)
     )
@@
       (project "Oro Link rev2"
         (path "/e89dcd22-1250-4a5b-b778-1c95a0dd623d/a5104146-06a0-496e-bda0-1e4731a261c3"
-          (reference "#PWR062") (unit 1)
+          (reference "#PWR0107") (unit 1)
         )
       )
@@
         )
         (path "/e89dcd22-1250-4a5b-b778-1c95a0dd623d/a5104146-06a0-496e-bda0-1e4731a261c3"
-          (reference "#PWR069") (unit 1)
+          (reference "#PWR0114") (unit 1)
         )
       )
@@
         )
         (path "/e89dcd22-1250-4a5b-b778-1c95a0dd623d/a5104146-06a0-496e-bda0-1e4731a261c3"
-          (reference "#PWR071") (unit 1)
+          (reference "#PWR0116") (unit 1)
         )
       )
@@
   (symbol (lib_id "SamacSys_Parts:UUP1H0R1MCL1GS") (at 80.01 132.08 0) (unit 1)
     (in_bom yes) (on_board yes) (dnp no)
-    (property "Reference" "C29" (at 91.44 133.35 0)
+    (property "Reference" "C57" (at 91.44 133.35 0)
       (effects (font (size 1.27 1.27)))
     )
@@
       (project "Oro Link rev2"
         (path "/e89dcd22-1250-4a5b-b778-1c95a0dd623d/a5104146-06a0-496e-bda0-1e4731a261c3"
-          (reference "C29") (unit 1)
+          (reference "C57") (unit 1)
         )
       )
@@
         )
         (path "/e89dcd22-1250-4a5b-b778-1c95a0dd623d/a5104146-06a0-496e-bda0-1e4731a261c3"
-          (reference "#PWR066") (unit 1)
+          (reference "#PWR0111") (unit 1)
         )
       )
@@
   (symbol (lib_id "power:+3V3") (at 104.14 74.93 0) (unit 1)
     (in_bom yes) (on_board yes) (dnp no) (fields_autoplaced)
-    (property "Reference" "#PWR063" (at 104.14 78.74 0)
+    (property "Reference" "#PWR0108" (at 104.14 78.74 0)
       (effects (font (size 1.27 1.27)) hide)
     )
@@
       (project "Oro Link rev2"
         (path "/e89dcd22-1250-4a5b-b778-1c95a0dd623d/a5104146-06a0-496e-bda0-1e4731a261c3"
-          (reference "#PWR063") (unit 1)
+          (reference "#PWR0108") (unit 1)
         )
       )
@@
   (symbol (lib_id "power:+3V3") (at 72.39 138.43 0) (unit 1)
     (in_bom yes) (on_board yes) (dnp no) (fields_autoplaced)
-    (property "Reference" "#PWR061" (at 72.39 142.24 0)
+    (property "Reference" "#PWR0106" (at 72.39 142.24 0)
       (effects (font (size 1.27 1.27)) hide)
     )
@@
       (project "Oro Link rev2"
         (path "/e89dcd22-1250-4a5b-b778-1c95a0dd623d/a5104146-06a0-496e-bda0-1e4731a261c3"
-          (reference "#PWR061") (unit 1)
+          (reference "#PWR0106") (unit 1)
         )
       )
@@
   (symbol (lib_id "SamacSys_Parts:UUP1H0R1MCL1GS") (at 80.01 113.03 0) (unit 1)
     (in_bom yes) (on_board yes) (dnp no)
-    (property "Reference" "C27" (at 91.44 114.3 0)
+    (property "Reference" "C55" (at 91.44 114.3 0)
       (effects (font (size 1.27 1.27)))
     )
@@
       (project "Oro Link rev2"
         (path "/e89dcd22-1250-4a5b-b778-1c95a0dd623d/a5104146-06a0-496e-bda0-1e4731a261c3"
-          (reference "C27") (unit 1)
+          (reference "C55") (unit 1)
         )
       )
@@
       (project "Oro Link rev2"
         (path "/e89dcd22-1250-4a5b-b778-1c95a0dd623d/a5104146-06a0-496e-bda0-1e4731a261c3"
-          (reference "J5") (unit 1)
+          (reference "J9") (unit 1)
         )
       )
@@
         )
         (path "/e89dcd22-1250-4a5b-b778-1c95a0dd623d/a5104146-06a0-496e-bda0-1e4731a261c3"
-          (reference "#PWR068") (unit 1)
+          (reference "#PWR0113") (unit 1)
         )
       )
@@
         )
         (path "/e89dcd22-1250-4a5b-b778-1c95a0dd623d/a5104146-06a0-496e-bda0-1e4731a261c3"
-          (reference "D7") (unit 1)
+          (reference "D14") (unit 1)
         )
       )
@@
         )
         (path "/e89dcd22-1250-4a5b-b778-1c95a0dd623d/a5104146-06a0-496e-bda0-1e4731a261c3"
-          (reference "#PWR070") (unit 1)
+          (reference "#PWR0115") (unit 1)
         )
       )
@@
   (symbol (lib_id "SamacSys_Parts:UUP1H0R1MCL1GS") (at 80.01 119.38 0) (unit 1)
     (in_bom yes) (on_board yes) (dnp no)
-    (property "Reference" "C28" (at 91.44 120.65 0)
+    (property "Reference" "C56" (at 91.44 120.65 0)
       (effects (font (size 1.27 1.27)))
     )
@@
       (project "Oro Link rev2"
         (path "/e89dcd22-1250-4a5b-b778-1c95a0dd623d/a5104146-06a0-496e-bda0-1e4731a261c3"
-          (reference "C28") (unit 1)
-        )
-      )
+          (reference "C56") (unit 1)
+        )
+      )

Commit message: first few boards laid out
Parts:
- renumbered C55 to C54, C56 to C55, C57 to C56, C58 to C57, C59 to C58, S2 to S3, S3 to S4
Changed lines of the file:
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@@
     (rev "2")
     (company "Oro Operating System")
+    (comment 1 "://oro.sh")
+    (comment 2 "Joshua Lee Junon")
   )
   (junction (at 165.1 80.01) (diameter 0) (color 0 0 0 0)
@@
   (symbol (lib_id "SamacSys_Parts:UUP1H0R1MCL1GS") (at 92.71 125.73 180) (unit 1)
     (in_bom yes) (on_board yes) (dnp no)
-    (property "Reference" "C59" (at 91.44 127 0)
+    (property "Reference" "C58" (at 91.44 127 0)
       (effects (font (size 1.27 1.27)))
     )
@@
       (project "Oro Link rev2"
         (path "/e89dcd22-1250-4a5b-b778-1c95a0dd623d/a5104146-06a0-496e-bda0-1e4731a261c3"
-          (reference "C59") (unit 1)
+          (reference "C58") (unit 1)
         )
       )
@@
   (symbol (lib_id "power:GND") (at 165.1 97.79 0) (unit 1)
     (in_bom yes) (on_board yes) (dnp no) (fields_autoplaced)
-    (property "Reference" "#PWR0110" (at 165.1 104.14 0)
+    (property "Reference" "#PWR0140" (at 165.1 104.14 0)
       (effects (font (size 1.27 1.27)) hide)
     )
@@
       (project "Oro Link rev2"
         (path "/e89dcd22-1250-4a5b-b778-1c95a0dd623d/a5104146-06a0-496e-bda0-1e4731a261c3"
-          (reference "#PWR0110") (unit 1)
+          (reference "#PWR0140") (unit 1)
         )
       )
@@
         )
         (path "/e89dcd22-1250-4a5b-b778-1c95a0dd623d/a5104146-06a0-496e-bda0-1e4731a261c3"
-          (reference "C60") (unit 1)
+          (reference "C59") (unit 1)
         )
       )
@@
   (symbol (lib_id "power:GND") (at 113.03 73.66 0) (unit 1)
     (in_bom yes) (on_board yes) (dnp no) (fields_autoplaced)
-    (property "Reference" "#PWR0109" (at 113.03 80.01 0)
+    (property "Reference" "#PWR0139" (at 113.03 80.01 0)
       (effects (font (size 1.27 1.27)) hide)
     )
@@
       (project "Oro Link rev2"
         (path "/e89dcd22-1250-4a5b-b778-1c95a0dd623d/a5104146-06a0-496e-bda0-1e4731a261c3"
-          (reference "#PWR0109") (unit 1)
+          (reference "#PWR0139") (unit 1)
         )
       )
@@
   (symbol (lib_id "SamacSys_Parts:UUP1H0R1MCL1GS") (at 80.01 138.43 0) (unit 1)
     (in_bom yes) (on_board yes) (dnp no)
-    (property "Reference" "C58" (at 91.44 139.7 0)
+    (property "Reference" "C57" (at 91.44 139.7 0)
       (effects (font (size 1.27 1.27)))
     )
@@
       (project "Oro Link rev2"
         (path "/e89dcd22-1250-4a5b-b778-1c95a0dd623d/a5104146-06a0-496e-bda0-1e4731a261c3"
-          (reference "C58") (unit 1)
+          (reference "C57") (unit 1)
         )
       )
@@
         )
         (path "/e89dcd22-1250-4a5b-b778-1c95a0dd623d/a5104146-06a0-496e-bda0-1e4731a261c3"
-          (reference "#PWR0112") (unit 1)
+          (reference "#PWR0142") (unit 1)
         )
       )
@@
   (symbol (lib_id "power:GND") (at 100.33 143.51 0) (unit 1)
     (in_bom yes) (on_board yes) (dnp no) (fields_autoplaced)
-    (property "Reference" "#PWR0107" (at 100.33 149.86 0)
+    (property "Reference" "#PWR0137" (at 100.33 149.86 0)
       (effects (font (size 1.27 1.27)) hide)
     )
@@
       (project "Oro Link rev2"
         (path "/e89dcd22-1250-4a5b-b778-1c95a0dd623d/a5104146-06a0-496e-bda0-1e4731a261c3"
-          (reference "#PWR0107") (unit 1)
+          (reference "#PWR0137") (unit 1)
         )
       )
@@
   (symbol (lib_id "SamacSys_Parts:206-124") (at 124.46 74.93 0) (unit 1)
     (in_bom yes) (on_board yes) (dnp no)
-    (property "Reference" "S2" (at 135.89 68.58 0)
+    (property "Reference" "S3" (at 135.89 68.58 0)
       (effects (font (size 1.27 1.27)))
     )
@@
       (project "Oro Link rev2"
         (path "/e89dcd22-1250-4a5b-b778-1c95a0dd623d/a5104146-06a0-496e-bda0-1e4731a261c3"
-          (reference "S2") (unit 1)
+          (reference "S3") (unit 1)
         )
       )
@@
         )
         (path "/e89dcd22-1250-4a5b-b778-1c95a0dd623d/a5104146-06a0-496e-bda0-1e4731a261c3"
-          (reference "#PWR0114") (unit 1)
+          (reference "#PWR0144") (unit 1)
         )
       )
@@
         )
         (path "/e89dcd22-1250-4a5b-b778-1c95a0dd623d/a5104146-06a0-496e-bda0-1e4731a261c3"
-          (reference "#PWR0116") (unit 1)
+          (reference "#PWR0146") (unit 1)
         )
       )
@@
   (symbol (lib_id "SamacSys_Parts:206-125") (at 168.91 74.93 0) (unit 1)
     (in_bom yes) (on_board yes) (dnp no)
-    (property "Reference" "S3" (at 180.34 68.58 0)
+    (property "Reference" "S4" (at 180.34 68.58 0)
       (effects (font (size 1.27 1.27)))
     )
@@
       (project "Oro Link rev2"
         (path "/e89dcd22-1250-4a5b-b778-1c95a0dd623d/a5104146-06a0-496e-bda0-1e4731a261c3"
-          (reference "S3") (unit 1)
+          (reference "S4") (unit 1)
         )
       )
@@
   (symbol (lib_id "SamacSys_Parts:UUP1H0R1MCL1GS") (at 80.01 132.08 0) (unit 1)
     (in_bom yes) (on_board yes) (dnp no)
-    (property "Reference" "C57" (at 91.44 133.35 0)
+    (property "Reference" "C56" (at 91.44 133.35 0)
       (effects (font (size 1.27 1.27)))
     )
@@
       (project "Oro Link rev2"
         (path "/e89dcd22-1250-4a5b-b778-1c95a0dd623d/a5104146-06a0-496e-bda0-1e4731a261c3"
-          (reference "C57") (unit 1)
+          (reference "C56") (unit 1)
         )
       )
@@
         )
         (path "/e89dcd22-1250-4a5b-b778-1c95a0dd623d/a5104146-06a0-496e-bda0-1e4731a261c3"
-          (reference "#PWR0111") (unit 1)
+          (reference "#PWR0141") (unit 1)
         )
       )
@@
   (symbol (lib_id "power:+3V3") (at 104.14 74.93 0) (unit 1)
     (in_bom yes) (on_board yes) (dnp no) (fields_autoplaced)
-    (property "Reference" "#PWR0108" (at 104.14 78.74 0)
+    (property "Reference" "#PWR0138" (at 104.14 78.74 0)
       (effects (font (size 1.27 1.27)) hide)
     )
@@
       (project "Oro Link rev2"
         (path "/e89dcd22-1250-4a5b-b778-1c95a0dd623d/a5104146-06a0-496e-bda0-1e4731a261c3"
-          (reference "#PWR0108") (unit 1)
+          (reference "#PWR0138") (unit 1)
         )
       )
@@
   (symbol (lib_id "power:+3V3") (at 72.39 138.43 0) (unit 1)
     (in_bom yes) (on_board yes) (dnp no) (fields_autoplaced)
-    (property "Reference" "#PWR0106" (at 72.39 142.24 0)
+    (property "Reference" "#PWR0136" (at 72.39 142.24 0)
       (effects (font (size 1.27 1.27)) hide)
     )
@@
       (project "Oro Link rev2"
         (path "/e89dcd22-1250-4a5b-b778-1c95a0dd623d/a5104146-06a0-496e-bda0-1e4731a261c3"
-          (reference "#PWR0106") (unit 1)
+          (reference "#PWR0136") (unit 1)
         )
       )
@@
   (symbol (lib_id "SamacSys_Parts:UUP1H0R1MCL1GS") (at 80.01 113.03 0) (unit 1)
     (in_bom yes) (on_board yes) (dnp no)
-    (property "Reference" "C55" (at 91.44 114.3 0)
+    (property "Reference" "C54" (at 91.44 114.3 0)
       (effects (font (size 1.27 1.27)))
     )
@@
       (project "Oro Link rev2"
         (path "/e89dcd22-1250-4a5b-b778-1c95a0dd623d/a5104146-06a0-496e-bda0-1e4731a261c3"
-          (reference "C55") (unit 1)
+          (reference "C54") (unit 1)
         )
       )
@@
       (project "Oro Link rev2"
         (path "/e89dcd22-1250-4a5b-b778-1c95a0dd623d/a5104146-06a0-496e-bda0-1e4731a261c3"
-          (reference "J9") (unit 1)
+          (reference "J27") (unit 1)
         )
       )
@@
         )
         (path "/e89dcd22-1250-4a5b-b778-1c95a0dd623d/a5104146-06a0-496e-bda0-1e4731a261c3"
-          (reference "#PWR0113") (unit 1)
+          (reference "#PWR0143") (unit 1)
         )
       )
@@
         )
         (path "/e89dcd22-1250-4a5b-b778-1c95a0dd623d/a5104146-06a0-496e-bda0-1e4731a261c3"
-          (reference "D14") (unit 1)
+          (reference "D11") (unit 1)
         )
       )
@@
         )
         (path "/e89dcd22-1250-4a5b-b778-1c95a0dd623d/a5104146-06a0-496e-bda0-1e4731a261c3"
-          (reference "#PWR0115") (unit 1)
+          (reference "#PWR0145") (unit 1)
         )
       )
@@
   (symbol (lib_id "SamacSys_Parts:UUP1H0R1MCL1GS") (at 80.01 119.38 0) (unit 1)
     (in_bom yes) (on_board yes) (dnp no)
-    (property "Reference" "C56" (at 91.44 120.65 0)
+    (property "Reference" "C55" (at 91.44 120.65 0)
       (effects (font (size 1.27 1.27)))
     )
@@
       (project "Oro Link rev2"
         (path "/e89dcd22-1250-4a5b-b778-1c95a0dd623d/a5104146-06a0-496e-bda0-1e4731a261c3"
-          (reference "C56") (unit 1)
-        )
-      )
+          (reference "C55") (unit 1)
+        )
+      )

Commit message: first panelization of entire modular dev board
Parts:
- removed C30: 1nF 5kV, CAPC5664X270N, symbol SamacSys_Parts:HV2225Y102KXMATHV
Connections:
- net C1+: no longer C55.1, IC6.4 (C2+)
- net CTS: no longer S3.12, S3.9, S4.C2, S4.C3
- net RTS: no longer S3.10, S3.11, S4.D2, S4.D3
- net RX: no longer S3.14, S3.15, S4.B2, S4.B3
- net TX: no longer S3.13, S3.16, S4.A2, S4.A3
- new net C2+: C55.1, IC6.4 (C2+)
- new net D_CTS: S3.12, S3.9, S4.C2, S4.C3
- new net D_RTS: S3.10, S3.11, S4.D2, S4.D3
- new net D_RX: S3.14, S3.15, S4.B2, S4.B3
- new net D_TX: S3.13, S3.16, S4.A2, S4.A3
Other:
- moved on the sheet: C54, C55, C56, C57, C58, D6

Commit message: initial board layout
Parts:
- J2: value 855-M50-3500542 -> 67996-110HLF; footprint SamacSys_Parts:M503500542 -> HDRV10W67P254_2X5_1270X483X858P; symbol SamacSys_Parts:M50-3500542 -> SamacSys_Parts:67996-110HLF; Arrow Part Number (none) -> 67996-110HLF; Arrow Price/Stock (none) -> https://www.arrow.com/en/products/67996-110hlf/amphenol-fci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; Height 4.15 -> 8.58; Manufacturer_Name Harwin -> Amphenol Communications Solutions; Manufacturer_Part_Number M50-3500542 -> 67996-110HLF; Mouser Part Number 855-M50-3500542 -> 649-67996-110HLF; Mouser Price/Stock https://www.mouser.co.uk/ProductDetail/Harwin/M50-3500542?q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 -> https://www.mouser.co.uk/ProductDetail/Amphenol-FCI/67996-1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
- renumbered C54 to C46, C55 to C47, C56 to C48, C57 to C49, C58 to C50
