File: OroLink.kicad_pcb (KiCad board)
At the start: 4 copper layers, 112.8 x 65 mm, 182 parts, among them IC1 STM32F479VGT6, IC2 TPS73733DCQ, IC3 TPS6734IDR, IC4 ENC28J60-I_SO, IC5 ENC28J60-I_SO, IC6 SN75C3232EPWR, IC7 IS31FL3218-GRLS2, J1 67996-408HLF, J2 DF63-5P-3.96DSA, J3 67996-408HLF, J4 3-2328724-1, J5 JXD2-0Z10NL, J6 JXD2-0Z10NL, J7 OroConn6p, Q1 PMV20ENR, Q2 PMV20ENR, Q3 PMV20ENR, T1 PT61017XPEL, T2 PT61017XPEL, X1 7P-26.000MBP-T, Y1 25MHz, Y2 25MHz

Commit message: minor PCB tweaks
Parts:
- moved G*** 221.4 mm to (162.1, 73.7)
- moved DBG30 23.8 mm to (180.8, 66.5)
- moved DBG31 0.20 mm to (180.8, 65.0)
- moved DBG34 0.15 mm to (180.8, 63.4)
- moved DBG32 0.10 mm to (180.8, 61.8)
- moved DBG33 0.05 mm to (180.8, 60.2)
Changed lines of the file:
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@@
   )
   (footprint "Oro Footprints:DebugPin" (layer "F.Cu")
-    (at 180.848 63.246)
+    (at 180.848 63.3984)
     (property "Sheetfile" "power-supply.kicad_sch")
     (property "Sheetname" "Power Supply")
@@
   )
   (footprint "Oro Footprints:DebugPin" (layer "F.Cu")
-    (at 180.848 64.77)
+    (at 180.848 64.9732)
     (property "Sheetfile" "power-supply.kicad_sch")
     (property "Sheetname" "Power Supply")
@@
   )
   (footprint "Oro Footprints:DebugPin" (layer "F.Cu")
-    (at 180.848 60.198)
+    (at 180.848 60.2488)
     (property "Sheetfile" "power-supply.kicad_sch")
     (property "Sheetname" "Power Supply")
@@
   )
   (footprint "Oro Footprints:DebugPin" (layer "F.Cu")
-    (at 195.834 85.09)
+    (at 180.848 66.548)
     (property "Sheetfile" "power-supply.kicad_sch")
     (property "Sheetname" "Power Supply")
@@
   )
   (footprint "Oro Footprints:DebugPin" (layer "F.Cu")
-    (at 180.848 61.722)
+    (at 180.848 61.8236)
     (property "Sheetfile" "power-supply.kicad_sch")
     (property "Sheetname" "Power Supply")
@@
   )
   (footprint "LOGO" (layer "B.Cu")
-    (at -55.9672 35.276153 180)
+    (at 162.052 73.66 180)
     (attr board_only exclude_from_pos_files exclude_from_bom)
     (fp_text reference "G***" (at 0 0) (layer "B.SilkS") hide
@@
     )
   )
-  (gr_rect (start -100.584 18.288) (end -39.37 38.354)
+  (gr_rect (start 141.6812 54.2544) (end 202.8952 74.3204)
     (stroke (width 0.15) (type default)) (fill none) (layer "F.SilkS"))
   (gr_line (start 29.625142 153.636) (end 150.432289 153.636)

Commit message: initial layout of components on rev4 board
Parts:
- removed DBG1, DBG10, DBG11, DBG12, DBG13, DBG14, DBG15, DBG16, DBG17, DBG18, DBG19, DBG2, DBG20, DBG21, DBG22, DBG23, DBG24, DBG25, DBG26, DBG27, DBG28, DBG29, DBG3, DBG30, DBG31, DBG32, DBG33, DBG34, DBG35, DBG36, DBG37, DBG38, DBG39, DBG4, DBG40, DBG41, DBG42, DBG43, DBG44, DBG45, DBG5, DBG6, DBG7, DBG8, DBG9: ~, Oro Footprints:DebugPin
- C31, C40, D12, D14: moved to B.Cu
- C33, C35, C44, IC2, R14, R15, R16, R17, R20, R25, R26, R27, R28, R9, S1, X1: moved to F.Cu
- moved R21 338.7 mm to (173.6, 101.4), turned to -90 degrees
- moved R22 336.6 mm to (171.8, 101.4), turned to -90 degrees
- moved R24 334.3 mm to (170.0, 101.4), turned to -90 degrees
- moved R23 332.8 mm to (168.2, 101.4), turned to -90 degrees
- moved R28 322.0 mm to (191.4, 96.8)
- moved R10 321.2 mm to (129.5, 101.4), turned to -90 degrees
- moved R26 319.5 mm to (191.4, 94.3)
- moved R11 319.1 mm to (127.7, 101.4), turned to -90 degrees
- moved R12 317.1 mm to (125.9, 101.4), turned to -90 degrees
- moved R13 315.0 mm to (124.1, 101.4), turned to -90 degrees
- moved R27 313.8 mm to (184.3, 96.8), turned to 90 degrees
- moved R25 313.4 mm to (184.3, 94.3), turned to -90 degrees
- moved C40 309.4 mm to (187.8, 90.1), turned to -90 degrees
- moved C39 289.9 mm to (172.7, 102.1), turned to -90 degrees
- moved FB3 288.1 mm to (170.9, 103.7), turned to 90 degrees
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Connections:
- D4 pad 4: /System Ethernet/TX+ -> /System Ethernet/TX-
- D4 pad 5: /System Ethernet/TX- -> /System Ethernet/TX+
- D8 pad 4: /External Ethernet/TX+ -> /External Ethernet/TX-
- D8 pad 5: /External Ethernet/TX- -> /External Ethernet/TX+
Other:
- outline, holes or cut-outs redrawn
- board text removed: "ORO OPERATING SYSTEM x86 link board v3.2023.04.05 oro.sh"
- board text removed: "オロ オペレーティング システム"

Commit message: add new board characteristics table
Other:
- board text added: "112.7500 mm x 65.0000 mm"
- board text removed: "121.9200 mm x 96.0120 mm"
- board text removed: "Yes"
