File: PCB/microcontroller.kicad_sch (KiCad schematic)
At the start: 25 parts, among them IC1 STM32F479VGT6, X1 7P-26.000MBP-T

Commit message: fix i2c pull-up resistor footprint mismatch
Parts:
- R1, R2: footprint RESC1005X40N -> RESC6431X65N; Height 0.4 -> 0.65; Manufacturer_Name MULTICOMP -> KEMET; Manufacturer_Part_Number MCWR04X4701FTL -> RC2512FK-074K7L
Changed lines of the file:
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@@
       (effects (font (size 1.27 1.27)) (justify right))
     )
-    (property "Footprint" "RESC1005X40N" (at 68.58 34.29 0)
-      (effects (font (size 1.27 1.27)) (justify left) hide)
-    )
-    (property "Datasheet" "https://componentsearchengine.com/Datasheets/2/MCWR04X4701FTL.pdf" (at 71.12 34.29 0)
-      (effects (font (size 1.27 1.27)) (justify left) hide)
-    )
-    (property "Description" "MULTICOMP - MCWR04X4701FTL - RES, 4K7, 1%, 0.0625W, 0402, THICK FILM" (at 73.66 34.29 0)
-      (effects (font (size 1.27 1.27)) (justify left) hide)
-    )
-    (property "Height" "0.4" (at 76.2 34.29 0)
-      (effects (font (size 1.27 1.27)) (justify left) hide)
-    )
-    (property "Manufacturer_Name" "MULTICOMP" (at 78.74 34.29 0)
-      (effects (font (size 1.27 1.27)) (justify left) hide)
-    )
-    (property "Manufacturer_Part_Number" "MCWR04X4701FTL" (at 81.28 34.29 0)
+    (property "Footprint" "RESC6431X65N" (at 68.58 34.29 0)
+      (effects (font (size 1.27 1.27)) (justify left) hide)
+    )
+    (property "Datasheet" "https://altium.componentsearchengine.com/Datasheets/2/RC2512FK-074K7L.pdf" (at 71.12 34.29 0)
+      (effects (font (size 1.27 1.27)) (justify left) hide)
+    )
+    (property "Description" "YAGEO - RC2512FK-074K7L - SMD Chip Resistor, 2512 [6432 Metric], 4.7 kohm, RC Series, 200 V, Thick Film, 1 W" (at 73.66 34.29 0)
+      (effects (font (size 1.27 1.27)) (justify left) hide)
+    )
+    (property "Height" "0.65" (at 76.2 34.29 0)
+      (effects (font (size 1.27 1.27)) (justify left) hide)
+    )
+    (property "Manufacturer_Name" "KEMET" (at 78.74 34.29 0)
+      (effects (font (size 1.27 1.27)) (justify left) hide)
+    )
+    (property "Manufacturer_Part_Number" "RC2512FK-074K7L" (at 81.28 34.29 0)
       (effects (font (size 1.27 1.27)) (justify left) hide)
     )
@@
       (effects (font (size 1.27 1.27)) (justify right))
     )
-    (property "Footprint" "RESC1005X40N" (at 59.69 34.29 0)
-      (effects (font (size 1.27 1.27)) (justify left) hide)
-    )
-    (property "Datasheet" "https://componentsearchengine.com/Datasheets/2/MCWR04X4701FTL.pdf" (at 62.23 34.29 0)
-      (effects (font (size 1.27 1.27)) (justify left) hide)
-    )
-    (property "Description" "MULTICOMP - MCWR04X4701FTL - RES, 4K7, 1%, 0.0625W, 0402, THICK FILM" (at 64.77 34.29 0)
-      (effects (font (size 1.27 1.27)) (justify left) hide)
-    )
-    (property "Height" "0.4" (at 67.31 34.29 0)
-      (effects (font (size 1.27 1.27)) (justify left) hide)
-    )
-    (property "Manufacturer_Name" "MULTICOMP" (at 69.85 34.29 0)
-      (effects (font (size 1.27 1.27)) (justify left) hide)
-    )
-    (property "Manufacturer_Part_Number" "MCWR04X4701FTL" (at 72.39 34.29 0)
-      (effects (font (size 1.27 1.27)) (justify left) hide)
-    )
+    (property "Footprint" "RESC6431X65N" (at 59.69 34.29 0)
+      (effects (font (size 1.27 1.27)) (justify left) hide)
+    )
+    (property "Datasheet" "https://altium.componentsearchengine.com/Datasheets/2/RC2512FK-074K7L.pdf" (at 62.23 34.29 0)
+      (effects (font (size 1.27 1.27)) (justify left) hide)
+    )
+    (property "Description" "YAGEO - RC2512FK-074K7L - SMD Chip Resistor, 2512 [6432 Metric], 4.7 kohm, RC Series, 200 V, Thick Film, 1 W" (at 64.77 34.29 0)
+      (effects (font (size 1.27 1.27)) (justify left) hide)
+    )
+    (property "Height" "0.65" (at 67.31 34.29 0)
+      (effects (font (size 1.27 1.27)) (justify left) hide)
+    )
+    (property "Manufacturer_Name" "KEMET" (at 69.85 34.29 0)
+      (effects (font (size 1.27 1.27)) (justify left) hide)
+    )
+    (property "Manufacturer_Part_Number" "RC2512FK-074K7L" (at 72.39 34.29 0)
+      (effects (font (size 1.27 1.27)) (justify left) hide)
+    )

Commit message: switch MCU debug LED to direct drive (closes #7)
Connections:
- net +3V3: no longer LED5.2
- net GND: now also LED5.1
- net at R5.2: now also LED5.2; no longer LED5.1
Changed lines of the file:
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@@
+    )
+  )
+  (symbol (lib_id "power:GND") (at 161.29 185.42 0) (mirror y) (unit 1)
+    (in_bom yes) (on_board yes) (dnp no) (fields_autoplaced)
+    (property "Reference" "#PWR069" (at 161.29 191.77 0)
+      (effects (font (size 1.27 1.27)) hide)
+    )
+    (property "Value" "GND" (at 161.29 189.5555 0)
+      (effects (font (size 1.27 1.27)))
+    )
+    (property "Footprint" "" (at 161.29 185.42 0)
+      (effects (font (size 1.27 1.27)) hide)
+    )
+    (property "Datasheet" "" (at 161.29 185.42 0)
+      (effects (font (size 1.27 1.27)) hide)
+    )
+    (pin "1")
+    (instances
+      (project "Oro Testbed v2"
+        (path "/3d0fc623-63eb-45e5-a304-e470d9b3a173"
+          (reference "#PWR069") (unit 1)
+        )
+      )
+      (project "OroLink"
+        (path "/e89dcd22-1250-4a5b-b778-1c95a0dd623d/dd173832-34f8-47c0-be66-f527d6e2d134"
+          (reference "#PWR09") (unit 1)
+        )
+      )
     )
   )
@@
         (path "/e89dcd22-1250-4a5b-b778-1c95a0dd623d/dd173832-34f8-47c0-be66-f527d6e2d134"
           (reference "S1") (unit 1)
-        )
-      )
-    )
-  )
-  (symbol (lib_id "power:+3V3") (at 161.29 185.42 0) (unit 1)
-    (in_bom yes) (on_board yes) (dnp no) (fields_autoplaced)
-    (property "Reference" "#PWR09" (at 161.29 189.23 0)
-      (effects (font (size 1.27 1.27)) hide)
-    )
-    (property "Value" "+3V3" (at 161.29 181.9181 0)
-      (effects (font (size 1.27 1.27)))
-    )
-    (property "Footprint" "" (at 161.29 185.42 0)
-      (effects (font (size 1.27 1.27)) hide)
-    )
-    (property "Datasheet" "" (at 161.29 185.42 0)
-      (effects (font (size 1.27 1.27)) hide)
-    )
-    (pin "1")
-    (instances
-      (project "OroLink"
-        (path "/e89dcd22-1250-4a5b-b778-1c95a0dd623d/dd173832-34f8-47c0-be66-f527d6e2d134"
-          (reference "#PWR09") (unit 1)
         )
       )
@@
     )
   )
-  (symbol (lib_id "SamacSys_Parts:AA3528VRVFS_A") (at 142.24 185.42 0) (unit 1)
+  (symbol (lib_id "SamacSys_Parts:AA3528VRVFS_A") (at 157.48 185.42 0) (mirror y) (unit 1)
     (in_bom yes) (on_board yes) (dnp no)
     (property "Reference" "LED5" (at 149.86 176.53 0)
@@
       (effects (font (size 1.27 1.27)) (justify top))
     )
-    (property "Footprint" "SamacSys_Parts:AA3528VRVFSA" (at 154.94 181.61 0)
+    (property "Footprint" "SamacSys_Parts:AA3528VRVFSA" (at 144.78 181.61 0)
       (effects (font (size 1.27 1.27)) (justify left bottom) hide)
     )
-    (property "Datasheet" "https://mouser.componentsearchengine.com/Datasheets/1/AA3528VRVFS_A.pdf" (at 154.94 184.15 0)
+    (property "Datasheet" "https://mouser.componentsearchengine.com/Datasheets/1/AA3528VRVFS_A.pdf" (at 144.78 184.15 0)
       (effects (font (size 1.27 1.27)) (justify left bottom) hide)
     )
-    (property "Description" "LED Uni-Color Violet 2-Pin SMD T/R" (at 154.94 186.69 0)
+    (property "Description" "LED Uni-Color Violet 2-Pin SMD T/R" (at 144.78 186.69 0)
       (effects (font (size 1.27 1.27)) (justify left bottom) hide)
     )
-    (property "Height" "2.1" (at 154.94 189.23 0)
+    (property "Height" "2.1" (at 144.78 189.23 0)
       (effects (font (size 1.27 1.27)) (justify left bottom) hide)
     )
-    (property "Manufacturer_Name" "Kingbright" (at 154.94 191.77 0)
+    (property "Manufacturer_Name" "Kingbright" (at 144.78 191.77 0)
       (effects (font (size 1.27 1.27)) (justify left bottom) hide)
     )
-    (property "Manufacturer_Part_Number" "AA3528VRVFS/A" (at 154.94 194.31 0)
+    (property "Manufacturer_Part_Number" "AA3528VRVFS/A" (at 144.78 194.31 0)
       (effects (font (size 1.27 1.27)) (justify left bottom) hide)
     )
-    (property "Mouser Part Number" "604-AA3528VRVFS/A" (at 154.94 196.85 0)
+    (property "Mouser Part Number" "604-AA3528VRVFS/A" (at 144.78 196.85 0)
       (effects (font (size 1.27 1.27)) (justify left bottom) hide)
     )
-    (property "Mouser Price/Stock" "https://www.mouser.co.uk/ProductDetail/Kingbright/AA3528VRVFS-A?qs=rY7msk5yxfb63mh907EyRA%3D%3D" (at 154.94 199.39 0)
+    (property "Mouser Price/Stock" "https://www.mouser.co.uk/ProductDetail/Kingbright/AA3528VRVFS-A?qs=rY7msk5yxfb63mh907EyRA%3D%3D" (at 144.78 199.39 0)
       (effects (font (size 1.27 1.27)) (justify left bottom) hide)
     )
-    (property "Arrow Part Number" "AA3528VRVFS/A" (at 154.94 201.93 0)
+    (property "Arrow Part Number" "AA3528VRVFS/A" (at 144.78 201.93 0)
       (effects (font (size 1.27 1.27)) (justify left bottom) hide)
     )
-    (property "Arrow Price/Stock" "https://www.arrow.com/en/products/aa3528vrvfsa/kingbright?region=nac" (at 154.94 204.47 0)
+    (property "Arrow Price/Stock" "https://www.arrow.com/en/products/aa3528vrvfsa/kingbright?region=nac" (at 144.78 204.47 0)
       (effects (font (size 1.27 1.27)) (justify left bottom) hide)
     )
-    (property "Mouser Testing Part Number" "" (at 154.94 207.01 0)
+    (property "Mouser Testing Part Number" "" (at 144.78 207.01 0)
       (effects (font (size 1.27 1.27)) (justify left bottom) hide)
     )
-    (property "Mouser Testing Price/Stock" "" (at 154.94 209.55 0)
+    (property "Mouser Testing Price/Stock" "" (at 144.78 209.55 0)
       (effects (font (size 1.27 1.27)) (justify left bottom) hide)
     )
-    (property "Note" "DEBUG LED" (at 148.59 190.5 0)
-      (effects (font (size 1.27 1.27)))
-    )
+    (property "Note" "DEBUG LED" (at 151.13 190.5 0)
+      (effects (font (size 1.27 1.27)))
+    )

Commit message: switch to self-contained magnetics ethernet jack (closes #28)
Connections:
- net EXTETH_XFRM_EN: now reaches IC1.1 (PE2)
- net SYSETH_XFRM_EN: now reaches IC1.35 (PE10)
- no-connect marks 41 -> 39
Changed lines of the file:
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@@
   (junction (at 242.57 102.87) (diameter 0) (color 0 0 0 0)
+  )
+  (junction (at 46.99 73.66) (diameter 0) (color 0 0 0 0)
   )
   (junction (at 236.22 38.735) (diameter 0) (color 0 0 0 0)
@@
   (no_connect (at 111.76 50.8))
   (no_connect (at 162.56 78.74))
-  (no_connect (at 116.84 147.32))
   (no_connect (at 119.38 147.32))
   (no_connect (at 124.46 50.8))
@@
   (no_connect (at 162.56 111.76))
   (no_connect (at 106.68 147.32))
-  (no_connect (at 86.36 68.58))
   (no_connect (at 129.54 50.8))
   (no_connect (at 162.56 96.52))
@@
     (stroke (width 0) (type default))
   )
+  (wire (pts (xy 46.99 73.66) (xy 46.99 83.82))
+    (stroke (width 0) (type default))
+  )
   (wire (pts (xy 52.07 49.53) (xy 60.96 49.53))
     (stroke (width 0) (type default))
@@
     (stroke (width 0) (type default))
   )
+  (wire (pts (xy 46.99 73.66) (xy 86.36 73.66))
+    (stroke (width 0) (type default))
+  )
   (wire (pts (xy 76.2 71.12) (xy 86.36 71.12))
     (stroke (width 0) (type default))
@@
     (stroke (width 0) (type default))
   )
+  (wire (pts (xy 116.84 147.32) (xy 116.84 158.75))
+    (stroke (width 0) (type default))
+  )
   (wire (pts (xy 76.2 124.46) (xy 86.36 124.46))
     (stroke (width 0) (type default))
@@
     (stroke (width 0) (type default))
   )
-  (wire (pts (xy 71.12 73.66) (xy 86.36 73.66))
-    (stroke (width 0) (type default))
-  )
   (wire (pts (xy 74.93 99.06) (xy 86.36 99.06))
     (stroke (width 0) (type default))
@@
     (stroke (width 0) (type default))
   )
+  (wire (pts (xy 74.93 68.58) (xy 86.36 68.58))
+    (stroke (width 0) (type default))
+  )
   (wire (pts (xy 214.63 76.835) (xy 223.52 76.835))
     (stroke (width 0) (type default))
@@
     (stroke (width 0) (type default))
   )
-  (wire (pts (xy 46.99 71.755) (xy 46.99 83.82))
+  (wire (pts (xy 46.99 71.755) (xy 46.99 73.66))
     (stroke (width 0) (type default))
   )
@@
     (effects (font (size 1.27 1.27)) (justify right))
   )
+  (hierarchical_label "SYSETH_XFRM_EN" (shape output) (at 116.84 158.75 270) (fields_autoplaced)
+    (effects (font (size 1.27 1.27)) (justify right))
+  )
   (hierarchical_label "OLED_MOSI" (shape output) (at 137.16 39.37 90) (fields_autoplaced)
     (effects (font (size 1.27 1.27)) (justify left))
@@
   )
   (hierarchical_label "DBGUART_RX" (shape input) (at 109.22 158.75 270) (fields_autoplaced)
+    (effects (font (size 1.27 1.27)) (justify right))
+  )
+  (hierarchical_label "EXTETH_XFRM_EN" (shape output) (at 74.93 68.58 180) (fields_autoplaced)
     (effects (font (size 1.27 1.27)) (justify right))
   )
@@
         )
       )
-    )
-  )
-  (symbol (lib_id "power:+3V3") (at 71.12 73.66 0) (unit 1)
-    (in_bom yes) (on_board yes) (dnp no) (fields_autoplaced)
-    (property "Reference" "#PWR08" (at 71.12 77.47 0)
-      (effects (font (size 1.27 1.27)) hide)
-    )
-    (property "Value" "+3V3" (at 71.12 70.1581 0)
-      (effects (font (size 1.27 1.27)))
-    )
-    (property "Footprint" "" (at 71.12 73.66 0)
-      (effects (font (size 1.27 1.27)) hide)
-    )
-    (property "Datasheet" "" (at 71.12 73.66 0)
-      (effects (font (size 1.27 1.27)) hide)
-    )
-    (pin "1")
-    (instances
-      (project "OroLink"
-        (path "/e89dcd22-1250-4a5b-b778-1c95a0dd623d/dd173832-34f8-47c0-be66-f527d6e2d134"
-          (reference "#PWR08") (unit 1)
-        )
-      )

Commit message: re-annotate schematic
Parts:
- renumbered C15 to C18, C5 to C8, C6 to C9
Changed lines of the file:
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@@
       (project "OroLink"
         (path "/e89dcd22-1250-4a5b-b778-1c95a0dd623d/dd173832-34f8-47c0-be66-f527d6e2d134"
-          (reference "#PWR09") (unit 1)
+          (reference "#PWR08") (unit 1)
         )
       )
@@
       (project "OroLink"
         (path "/e89dcd22-1250-4a5b-b778-1c95a0dd623d/dd173832-34f8-47c0-be66-f527d6e2d134"
-          (reference "#PWR018") (unit 1)
+          (reference "#PWR017") (unit 1)
         )
       )
@@
       (project "OroLink"
         (path "/e89dcd22-1250-4a5b-b778-1c95a0dd623d/dd173832-34f8-47c0-be66-f527d6e2d134"
-          (reference "#PWR017") (unit 1)
+          (reference "#PWR016") (unit 1)
         )
       )
@@
       (project "OroLink"
         (path "/e89dcd22-1250-4a5b-b778-1c95a0dd623d/dd173832-34f8-47c0-be66-f527d6e2d134"
-          (reference "C9") (unit 1)
+          (reference "C12") (unit 1)
         )
       )
@@
   (symbol (lib_id "SamacSys_Parts:CL10A225KP8NNNC") (at 205.74 127 0) (unit 1)
     (in_bom yes) (on_board yes) (dnp no)
-    (property "Reference" "C5" (at 208.28 128.27 0)
+    (property "Reference" "C8" (at 208.28 128.27 0)
       (effects (font (size 1.27 1.27)))
     )
@@
       (project "OroLink"
         (path "/e89dcd22-1250-4a5b-b778-1c95a0dd623d/dd173832-34f8-47c0-be66-f527d6e2d134"
-          (reference "C5") (unit 1)
+          (reference "C8") (unit 1)
         )
       )
@@
       (project "OroLink"
         (path "/e89dcd22-1250-4a5b-b778-1c95a0dd623d/dd173832-34f8-47c0-be66-f527d6e2d134"
-          (reference "C13") (unit 1)
+          (reference "C16") (unit 1)
         )
       )
@@
   (symbol (lib_id "power:+3V3") (at 242.57 100.33 0) (unit 1)
     (in_bom yes) (on_board yes) (dnp no) (fields_autoplaced)
-    (property "Reference" "#PWR015" (at 242.57 104.14 0)
+    (property "Reference" "#PWR014" (at 242.57 104.14 0)
       (effects (font (size 1.27 1.27)) hide)
     )
@@
       (project "OroLink"
         (path "/e89dcd22-1250-4a5b-b778-1c95a0dd623d/dd173832-34f8-47c0-be66-f527d6e2d134"
-          (reference "#PWR015") (unit 1)
+          (reference "#PWR014") (unit 1)
         )
       )
@@
       (project "OroLink"
         (path "/e89dcd22-1250-4a5b-b778-1c95a0dd623d/dd173832-34f8-47c0-be66-f527d6e2d134"
-          (reference "C14") (unit 1)
+          (reference "C17") (unit 1)
         )
       )
@@
         )
         (path "/e89dcd22-1250-4a5b-b778-1c95a0dd623d/dd173832-34f8-47c0-be66-f527d6e2d134"
-          (reference "C2") (unit 1)
+          (reference "C5") (unit 1)
         )
       )
@@
       (project "OroLink"
         (path "/e89dcd22-1250-4a5b-b778-1c95a0dd623d/dd173832-34f8-47c0-be66-f527d6e2d134"
-          (reference "C1") (unit 1)
+          (reference "C4") (unit 1)
         )
       )
@@
   (symbol (lib_id "power:+3V3") (at 205.74 100.33 0) (unit 1)
     (in_bom yes) (on_board yes) (dnp no) (fields_autoplaced)
-    (property "Reference" "#PWR010" (at 205.74 104.14 0)
+    (property "Reference" "#PWR09" (at 205.74 104.14 0)
       (effects (font (size 1.27 1.27)) hide)
     )
@@
       (project "OroLink"
         (path "/e89dcd22-1250-4a5b-b778-1c95a0dd623d/dd173832-34f8-47c0-be66-f527d6e2d134"
-          (reference "#PWR010") (unit 1)
+          (reference "#PWR09") (unit 1)
         )
       )
@@
         )
         (path "/e89dcd22-1250-4a5b-b778-1c95a0dd623d/dd173832-34f8-47c0-be66-f527d6e2d134"
-          (reference "C17") (unit 1)
+          (reference "C20") (unit 1)
         )
       )
@@
       (project "OroLink"
         (path "/e89dcd22-1250-4a5b-b778-1c95a0dd623d/dd173832-34f8-47c0-be66-f527d6e2d134"
-          (reference "C12") (unit 1)
+          (reference "C15") (unit 1)
         )
       )
@@
       (project "OroLink"
         (path "/e89dcd22-1250-4a5b-b778-1c95a0dd623d/dd173832-34f8-47c0-be66-f527d6e2d134"
-          (reference "#PWR014") (unit 1)
+          (reference "#PWR013") (unit 1)
         )
       )
@@
   (symbol (lib_id "power:+3V3") (at 242.57 124.46 0) (unit 1)
     (in_bom yes) (on_board yes) (dnp no) (fields_autoplaced)
-    (property "Reference" "#PWR016" (at 242.57 128.27 0)
+    (property "Reference" "#PWR015" (at 242.57 128.27 0)
       (effects (font (size 1.27 1.27)) hide)
     )
@@
       (project "OroLink"
         (path "/e89dcd22-1250-4a5b-b778-1c95a0dd623d/dd173832-34f8-47c0-be66-f527d6e2d134"
-          (reference "#PWR016") (unit 1)
+          (reference "#PWR015") (unit 1)
         )
       )
@@
       (project "OroLink"
         (path "/e89dcd22-1250-4a5b-b778-1c95a0dd623d/dd173832-34f8-47c0-be66-f527d6e2d134"
-          (reference "#PWR011") (unit 1)
+          (reference "#PWR010") (unit 1)
         )
       )
@@
       (project "OroLink"
         (path "/e89dcd22-1250-4a5b-b778-1c95a0dd623d/dd173832-34f8-47c0-be66-f527d6e2d134"
-          (reference "C10") (unit 1)
+          (reference "C13") (unit 1)
         )
       )
@@
   (symbol (lib_id "SamacSys_Parts:CL10A225KP8NNNC") (at 205.74 133.35 0) (unit 1)
     (in_bom yes) (on_board yes) (dnp no)
-    (property "Reference" "C6" (at 208.28 134.62 0)
+    (property "Reference" "C9" (at 208.28 134.62 0)
       (effects (font (size 1.27 1.27)))
     )
@@
       (project "OroLink"
         (path "/e89dcd22-1250-4a5b-b778-1c95a0dd623d/dd173832-34f8-47c0-be66-f527d6e2d134"
-          (reference "C6") (unit 1)
+          (reference "C9") (unit 1)
         )
       )
@@
       (project "OroLink"
         (path "/e89dcd22-1250-4a5b-b778-1c95a0dd623d/dd173832-34f8-47c0-be66-f527d6e2d134"
-          (reference "C7") (unit 1)
+          (reference "C10") (unit 1)
         )
       )
@@
       (project "OroLink"
         (path "/e89dcd22-1250-4a5b-b778-1c95a0dd623d/dd173832-34f8-47c0-be66-f527d6e2d134"
-          (reference "C3") (unit 1)
+          (reference "C6") (unit 1)
         )
       )
@@
       (project "OroLink"
         (path "/e89dcd22-1250-4a5b-b778-1c95a0dd623d/dd173832-34f8-47c0-be66-f527d6e2d134"
-          (reference "C11") (unit 1)
+          (reference "C14") (unit 1)
         )
       )
@@
         )
         (path "/e89dcd22-1250-4a5b-b778-1c95a0dd623d/dd173832-34f8-47c0-be66-f527d6e2d134"
-          (reference "C4") (unit 1)
+          (reference "C7") (unit 1)
         )
       )
@@
       (project "OroLink"
         (path "/e89dcd22-1250-4a5b-b778-1c95a0dd623d/dd173832-34f8-47c0-be66-f527d6e2d134"
-          (reference "C8") (unit 1)
+          (reference "C11") (unit 1)
         )
       )
@@
       (project "OroLink"
         (path "/e89dcd22-1250-4a5b-b778-1c95a0dd623d/dd173832-34f8-47c0-be66-f527d6e2d134"
-          (reference "#PWR012") (unit 1)
+          (reference "#PWR011") (unit 1)
         )
       )
@@
   (symbol (lib_id "SamacSys_Parts:CL10A225KP8NNNC") (at 242.57 105.41 0) (unit 1)
     (in_bom yes) (on_board yes) (dnp no)
-    (property "Reference" "C15" (at 245.11 106.68 0)
+    (property "Reference" "C18" (at 245.11 106.68 0)
       (effects (font (size 1.27 1.27)))
     )
@@
       (project "OroLink"
         (path "/e89dcd22-1250-4a5b-b778-1c95a0dd623d/dd173832-34f8-47c0-be66-f527d6e2d134"
-          (reference "C15") (unit 1)
+          (reference "C18") (unit 1)
         )
       )
@@
       (project "OroLink"
         (path "/e89dcd22-1250-4a5b-b778-1c95a0dd623d/dd173832-34f8-47c0-be66-f527d6e2d134"
-          (reference "C16") (unit 1)
+          (reference "C19") (unit 1)
         )
       )
@@
   (symbol (lib_id "power:+3V3") (at 223.52 28.575 0) (unit 1)
     (in_bom yes) (on_board yes) (dnp no) (fields_autoplaced)
-    (property "Reference" "#PWR013" (at 223.52 32.385 0)
+    (property "Reference" "#PWR012" (at 223.52 32.385 0)
       (effects (font (size 1.27 1.27)) hide)
     )
@@
       (project "OroLink"
         (path "/e89dcd22-1250-4a5b-b778-1c95a0dd623d/dd173832-34f8-47c0-be66-f527d6e2d134"
-          (reference "#PWR013") (unit 1)
-        )
-      )
+          (reference "#PWR012") (unit 1)
+        )
+      )

Commit message: add pullup/down resistors and fix oro 6p lines with boot1/0
closes #24
closes #21
closes #15
closes #12
closes #6
closes #3
Parts:
- added R10 (x2): 10k, SamacSys_Parts:RESC5025X65N, symbol SamacSys_Parts:RC2010JK-0710KL
- renumbered R1 to R2, R2 to R3
Connections:
- net +3V3: now also R10.1
- net GND: now also R10.1
- net at C16.1, IC1.11 (NRST), S1.2 (NO): now also R10.2
- net BOOT1: now reaches IC1.31 (PB2)
- net BOOT1: now also R10.2
- net ~{FLASH} renamed BOOT0
- no-connect marks 39 -> 38
Other:
- moved on the sheet: C16, C21, S1

Commit message: replace 0.1u caps with larger package (closes #2)
Parts:
- C16: footprint SamacSys_Parts:CAPC0402X22N -> CAPC1005X33N; symbol SamacSys_Parts:GRT31C5C1H104FA02L -> SamacSys_Parts:MSAST1L3YB5104KFNA01; Arrow Part Number 01016D104KAT2A -> (none); Arrow Price/Stock https://www.arrow.com/en/products/01016d104kat2a/avx -> (none); Height 0.22 -> 0.33; Manufacturer_Name AVX -> TAIYO YUDEN; Manufacturer_Part_Number 01016D104KAT2A -> MSAST1L3YB5104KFNA01; Mouser Part Number 581-01016D104KAT2A -> (none); Mouser Price/Stock https://www.mouser.com/Search/Refine.aspx?Keyword=581-01016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 -> (none)
