File: PCB/indicator-lights.kicad_sch (KiCad schematic)
At the start: 10 parts, among them IC9 IS31FL3218-GRLS2

Commit message: replace remaining 0.1u caps with larger packages (ref #2)
Parts:
- C16: footprint SamacSys_Parts:CAPC0402X22N -> CAPC1005X33N; symbol SamacSys_Parts:01016D104KAT2A -> SamacSys_Parts:MSAST1L3YB5104KFNA01; Arrow Part Number 01016D104KAT2A -> (none); Arrow Price/Stock https://www.arrow.com/en/products/01016d104kat2a/avx -> (none); Height 0.22 -> 0.33; Manufacturer_Name AVX -> TAIYO YUDEN; Manufacturer_Part_Number 01016D104KAT2A -> MSAST1L3YB5104KFNA01; Mouser Part Number 581-01016D104KAT2A -> (none); Mouser Price/Stock https://www.mouser.com/Search/Refine.aspx?Keyword=581-01016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 -> (none)
Changed lines of the file:
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@@
     )
   )
-  (symbol (lib_id "SamacSys_Parts:01016D104KAT2A") (at 72.39 96.52 90) (mirror x) (unit 1)
+  (symbol (lib_id "SamacSys_Parts:MSAST1L3YB5104KFNA01") (at 72.39 96.52 90) (mirror x) (unit 1)
     (in_bom yes) (on_board yes) (dnp no)
     (property "Reference" "C16" (at 73.66 100.33 90)
@@
       (effects (font (size 1.27 1.27)) (justify right top))
     )
-    (property "Footprint" "SamacSys_Parts:CAPC0402X22N" (at 71.12 105.41 0)
+    (property "Footprint" "CAPC1005X33N" (at 71.12 105.41 0)
       (effects (font (size 1.27 1.27)) (justify left) hide)
     )
-    (property "Datasheet" "https://altium.componentsearchengine.com/Datasheets/1/01016D104KAT2A.pdf" (at 73.66 105.41 0)
+    (property "Datasheet" "https://www.mouser.de/datasheet/2/396/TaiyoYuden_MSAST1L3YB5104KFNA01_SS-3009733.pdf" (at 73.66 105.41 0)
       (effects (font (size 1.27 1.27)) (justify left) hide)
     )
-    (property "Description" "Multilayer Ceramic Capacitors MLCC - SMD/SMT 6.3V .1uF X5R 0101 10%" (at 76.2 105.41 0)
+    (property "Description" "Multilayer Ceramic Capacitors MLCC - SMD/SMT 0402 25VDC 0.1uF 10% X5R" (at 76.2 105.41 0)
       (effects (font (size 1.27 1.27)) (justify left) hide)
     )
-    (property "Height" "0.22" (at 78.74 105.41 0)
+    (property "Height" "0.33" (at 78.74 105.41 0)
       (effects (font (size 1.27 1.27)) (justify left) hide)
     )
-    (property "Manufacturer_Name" "AVX" (at 81.28 105.41 0)
+    (property "Manufacturer_Name" "TAIYO YUDEN" (at 81.28 105.41 0)
       (effects (font (size 1.27 1.27)) (justify left) hide)
     )
-    (property "Manufacturer_Part_Number" "01016D104KAT2A" (at 83.82 105.41 0)
+    (property "Manufacturer_Part_Number" "MSAST1L3YB5104KFNA01" (at 83.82 105.41 0)
       (effects (font (size 1.27 1.27)) (justify left) hide)
     )
-    (property "Mouser Part Number" "581-01016D104KAT2A" (at 86.36 105.41 0)
+    (property "Mouser Part Number" "" (at 86.36 105.41 0)
       (effects (font (size 1.27 1.27)) (justify left) hide)
     )
-    (property "Mouser Price/Stock" "https://www.mouser.com/Search/Refine.aspx?Keyword=581-01016D104KAT2A" (at 88.9 105.41 0)
+    (property "Mouser Price/Stock" "" (at 88.9 105.41 0)
       (effects (font (size 1.27 1.27)) (justify left) hide)
     )
-    (property "Arrow Part Number" "01016D104KAT2A" (at 91.44 105.41 0)
+    (property "Arrow Part Number" "" (at 91.44 105.41 0)
       (effects (font (size 1.27 1.27)) (justify left) hide)
     )
-    (property "Arrow Price/Stock" "https://www.arrow.com/en/products/01016d104kat2a/avx" (at 93.98 105.41 0)
+    (property "Arrow Price/Stock" "" (at 93.98 105.41 0)
       (effects (font (size 1.27 1.27)) (justify left) hide)
     )
