File: PCB/OroLink.kicad_pcb (KiCad board)
At the start: 4 copper layers, 114.9 x 65.4 mm, 161 parts, among them IC1 STM32F479VGT6, IC2 TPS73733DCQ, IC3 TPS6734IDR, IC4 ENC28J60-I_SO, IC5 ENC28J60-I_SO, IC6 SN75C3232EPWR, IC7 IS31FL3218-GRLS2, J1 67996-408HLF, J2 DF63-5P-3.96DSA, J3 67996-408HLF, J4 3-2328724-1, J5 JXD2-0Z10NL, J6 JXD2-0Z10NL, J7 OroConn6p, Q1 PMV20ENR, Q2 PMV20ENR, Q3 PMV20ENR, T1 PT61017XPEL, T2 PT61017XPEL, X1 7P-26.000MBP-T, Y1 25MHz, Y2 25MHz

Commit message: all but ethernet laid out
Parts:
- removed the C35 at (108.2, 89.3)
- removed the C45 at (191.8, 88.8)
- removed D10, D11, D4, D5, D6, D7, D8, D9: ESDS302DBVR, SamacSys_Parts:SOT95P280X145-5N
- removed D12: RFU02VSM8STR, SamacSys_Parts:SODFL2514X80N
- removed D13, D15: RCLAMP3552T.TNT, SamacSys_Parts:RCLAMP3552TTNT
- removed D14: P6SMB15A-Q, SamacSys_Parts:DIOM5436X244N
- removed DBG39: ~, Oro Footprints:DebugPin
- removed the R29 at (189.1, 103.6)
- removed T1, T2: PT61017XPEL, SamacSys_Parts:SOIC127P930X570-16N
- added C1: 1nF 5kV, SamacSys_Parts:CAPC4620X220N, F.Cu at (49.6, 43.2)
- added C2: 1nF 5kV, SamacSys_Parts:CAPC4620X220N, F.Cu at (49.6, 46.8)
- added C3: 1nF 5kV, SamacSys_Parts:CAPC4620X220N, F.Cu at (49.6, 50.5)
- added C41: 0.1u, SamacSys_Parts:CAPC1005X33N, F.Cu at (29.7, 66.2)
- added C44: 10u, SamacSys_Parts:CAPC2012X135N, F.Cu at (30.5, 64.0)
- added C52: 0.1u, SamacSys_Parts:CAPC1005X33N, F.Cu at (29.7, 94.0)
- added C55: 10u, SamacSys_Parts:CAPC2012X135N, F.Cu at (30.5, 91.8)
- added DBG10: ~, Oro Footprints:DebugPin, F.Cu at (50.6, 76.5)
- added DBG11: ~, Oro Footprints:DebugPin, F.Cu at (50.6, 78.6)
- added DBG12: ~, Oro Footprints:DebugPin, F.Cu at (18.5, 63.6)
- added DBG13: ~, Oro Footprints:DebugPin, F.Cu at (18.5, 65.7)
- added DBG14: ~, Oro Footprints:DebugPin, F.Cu at (20.6, 63.6)
- added DBG15: ~, Oro Footprints:DebugPin, F.Cu at (20.6, 65.7)
- added DBG16: ~, Oro Footprints:DebugPin, F.Cu at (22.7, 63.6)
- added DBG17: ~, Oro Footprints:DebugPin, F.Cu at (22.7, 65.7)
- added DBG18: ~, Oro Footprints:DebugPin, F.Cu at (18.5, 91.4)
- added DBG19: ~, Oro Footprints:DebugPin, F.Cu at (18.5, 93.5)
- added DBG20: ~, Oro Footprints:DebugPin, F.Cu at (20.6, 91.4)
- added DBG21: ~, Oro Footprints:DebugPin, F.Cu at (20.6, 93.5)
- added DBG22: ~, Oro Footprints:DebugPin, F.Cu at (22.7, 91.4)
- added DBG23: ~, Oro Footprints:DebugPin, F.Cu at (22.7, 93.5)
- added DBG28: ~, Oro Footprints:DebugPin, F.Cu at (52.6, 55.3)
- added DBG29: ~, Oro Footprints:DebugPin, F.Cu at (52.6, 61.6)
- added DBG30: ~, Oro Footprints:DebugPin, F.Cu at (52.6, 63.7)
- added DBG31: ~, Oro Footprints:DebugPin, F.Cu at (210.8, 75.7)
- added DBG32: ~, Oro Footprints:DebugPin, F.Cu at (212.3, 75.7)
- added DBG7: ~, Oro Footprints:DebugPin, F.Cu at (50.6, 70.2)
- added DBG8: ~, Oro Footprints:DebugPin, F.Cu at (50.6, 72.3)
- added DBG9: ~, Oro Footprints:DebugPin, F.Cu at (50.6, 74.4)
- added IC5: PMV20ENR, SamacSys_Parts:SOT95P230X110-3N, F.Cu at (122.2, 86.7)
- added IC7: PMV20ENR, SamacSys_Parts:SOT95P230X110-3N, F.Cu at (26.1, 92.7)
- added R1: 10k, SamacSys_Parts:RESC1005X40N, F.Cu at (128.4, 79.9)
- added R11: 10k, SamacSys_Parts:RESC1005X40N, F.Cu at (157.9, 102.6)
- added R12: 10k, SamacSys_Parts:RESC1005X40N, F.Cu at (157.9, 103.6)
- added R18: 10k, SamacSys_Parts:RESC1005X40N, F.Cu at (114.6, 66.4)
- added R19: 10k, SamacSys_Parts:RESC1005X40N, F.Cu at (106.4, 51.3)
- added R20: 10k, SamacSys_Parts:RESC1005X40N, F.Cu at (115.7, 66.4)
- added R21: 10k, SamacSys_Parts:RESC1005X40N, F.Cu at (107.7, 51.3)
- added R22: 10k, SamacSys_Parts:RESC1005X40N, F.Cu at (112.6, 66.4)
- added R23: 10k, SamacSys_Parts:RESC1005X40N, F.Cu at (111.5, 66.4)
- added R25: 10k, SamacSys_Parts:RESC1005X40N, F.Cu at (102.6, 78.0)
- added R26: 10k, SamacSys_Parts:RESC1005X40N, F.Cu at (102.6, 81.7)
- added R39: 10k, SamacSys_Parts:RESC1005X40N, F.Cu at (42.6, 70.2)
- added R40: 10k, SamacSys_Parts:RESC1005X40N, F.Cu at (42.6, 72.4)
- added R41: 10k, SamacSys_Parts:RESC1005X40N, F.Cu at (42.6, 74.5)
- added R42: 10k, SamacSys_Parts:RESC1005X40N, F.Cu at (42.6, 76.7)
- added R44: 10k, SamacSys_Parts:RESC1005X40N, F.Cu at (42.6, 78.8)
- added R5: 10k, SamacSys_Parts:RESC1005X40N, F.Cu at (126.2, 86.1)
- added R7: 10k, SamacSys_Parts:RESC1005X40N, F.Cu at (151.8, 68.5)
- added R8: 10k, SamacSys_Parts:RESC1005X40N, F.Cu at (151.8, 67.3)
- C10: renamed from C7; footprint SamacSys_Parts:CAPC0402X22N -> SamacSys_Parts:CAPC1005X33N
- C11: renamed from C8; footprint SamacSys_Parts:CAPC0402X22N -> SamacSys_Parts:CAPC1005X33N
- C12: renamed from C9; footprint SamacSys_Parts:CAPC0402X22N -> SamacSys_Parts:CAPC1005X33N
- C13: renamed from C10; footprint SamacSys_Parts:CAPC0402X22N -> SamacSys_Parts:CAPC1005X33N
- C14: renamed from C11; footprint SamacSys_Parts:CAPC0402X22N -> SamacSys_Parts:CAPC1005X33N
- C15: renamed from C12; footprint SamacSys_Parts:CAPC0402X22N -> SamacSys_Parts:CAPC1005X33N
- C16: renamed from C13; footprint SamacSys_Parts:CAPC0402X22N -> SamacSys_Parts:CAPC1005X33N
- C17: renamed from C14; footprint SamacSys_Parts:CAPC0402X22N -> SamacSys_Parts:CAPC1005X33N
- C19: renamed from C16; footprint SamacSys_Parts:CAPC0402X22N -> SamacSys_Parts:CAPC1005X33N
- C36, C37, C38, C39, C40: footprint SamacSys_Parts:CAPC0402X22N -> SamacSys_Parts:CAPC1005X33N
- C4: renamed from C1; footprint SamacSys_Parts:CAPC0402X22N -> SamacSys_Parts:CAPC1005X33N
- C42: renamed from C33; footprint SamacSys_Parts:CAPC0402X22N -> SamacSys_Parts:CAPC1005X33N
- C43: renamed from C34; footprint SamacSys_Parts:CAPC0402X22N -> SamacSys_Parts:CAPC1005X33N
- C47: renamed from C46; footprint SamacSys_Parts:CAPC0402X22N -> SamacSys_Parts:CAPC1005X33N
- C48: renamed from C47; footprint SamacSys_Parts:CAPC0402X22N -> SamacSys_Parts:CAPC1005X33N
- C49: renamed from C48; footprint SamacSys_Parts:CAPC0402X22N -> SamacSys_Parts:CAPC1005X33N
- C50: renamed from C49; footprint SamacSys_Parts:CAPC0402X22N -> SamacSys_Parts:CAPC1005X33N
- C51: renamed from C50; footprint SamacSys_Parts:CAPC0402X22N -> SamacSys_Parts:CAPC1005X33N
- C53: renamed from C43; footprint SamacSys_Parts:CAPC0402X22N -> SamacSys_Parts:CAPC1005X33N
- C54: renamed from C44; footprint SamacSys_Parts:CAPC0402X22N -> SamacSys_Parts:CAPC1005X33N
- C59: renamed from C54; footprint SamacSys_Parts:CAPC0402X22N -> SamacSys_Parts:CAPC1005X33N
- C6: renamed from C3; footprint SamacSys_Parts:CAPC0402X22N -> SamacSys_Parts:CAPC1005X33N
- C61: renamed from C56; footprint SamacSys_Parts:CAPC0402X22N -> SamacSys_Parts:CAPC1005X33N
- D3: footprint SamacSys_Parts:DIOM5227X250N -> Oro Footprints:DIOM5227X250N
- IC3: value TPS6734IDR -> TPS6734ID
- J5, J6: value JXD2-0Z10NL -> 74990101241; footprint SamacSys_Parts:JXD20Z10NL -> Oro Footprints:74990101241
- R14: value 75R -> 510K; footprint SamacSys_Parts:RESC1005X40N -> SamacSys_Parts:RESC1608X55N
- R15, R16, R17, R27, R28, R30: value 75R -> 10k
- R2: renamed from R1; footprint SamacSys_Parts:RESC6431X65N -> SamacSys_Parts:RESC1005X40N; moved to F.Cu
- R24: renamed from R8; footprint SamacSys_Parts:RESC5025X65N -> SamacSys_Parts:RESC1005X40N
- R3: renamed from R2; footprint SamacSys_Parts:RESC6431X65N -> SamacSys_Parts:RESC1005X40N; moved to F.Cu
- R31: renamed from R10; footprint SamacSys_Parts:RESC0603X26N -> SamacSys_Parts:RESC1005X35N
- R32: renamed from R11; footprint SamacSys_Parts:RESC0603X26N -> SamacSys_Parts:RESC1005X35N
- R33: renamed from R12; footprint SamacSys_Parts:RESC0603X26N -> SamacSys_Parts:RESC1005X35N
- R34: renamed from R13; footprint SamacSys_Parts:RESC0603X26N -> SamacSys_Parts:RESC1005X35N
- R4: renamed from R3; footprint SamacSys_Parts:RESC5025X65N -> SamacSys_Parts:RESC1005X40N
- R45: renamed from R23; footprint SamacSys_Parts:RESC0603X26N -> SamacSys_Parts:RESC1005X35N
- R46: renamed from R24; footprint SamacSys_Parts:RESC0603X26N -> SamacSys_Parts:RESC1005X35N
- R47: renamed from R25; footprint SamacSys_Parts:RESC0603X26N -> SamacSys_Parts:RESC1005X35N
- R48: renamed from R26; footprint SamacSys_Parts:RESC0603X26N -> SamacSys_Parts:RESC1005X35N
- R54: renamed from R36; footprint SamacSys_Parts:RESC5025X65N -> SamacSys_Parts:RESC1005X40N
- R9: renamed from R5; footprint SamacSys_Parts:RESC5025X65N -> SamacSys_Parts:RESC1005X40N
- moved R28 91.6 mm to (102.6, 79.2), turned to 180 degrees
- moved C54 88.1 mm to (260.2, 102.3)
- moved FB3 88.1 mm to (258.4, 103.9)
- moved R46 88.1 mm to (261.1, 101.6)
- moved R45 88.1 mm to (259.3, 101.6)
- moved R47 88.1 mm to (255.8, 101.6)
- moved R48 88.1 mm to (257.6, 101.6)
- moved C53 88.1 mm to (256.7, 102.3)
- moved R27 87.6 mm to (102.6, 80.5)
- moved DBG24 79.4 mm to (37.3, 32.7)
- moved DBG25 79.4 mm to (38.7, 23.5)
- moved DBG27 79.4 mm to (53.2, 31.3)
- moved DBG26 79.4 mm to (53.3, 22.6)
- moved R30 73.0 mm to (121.6, 84.3)
- moved LED3 61.7 mm to (162.3, 107.4), turned to -90 degrees
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- renumbered C15 to C18, C17 to C20, C18 to C21, C19 to C22, C20 to C23, C21 to C24, C22 to C25, C23 to C26, C24 to C27, C25 to C28, C26 to C29, C27 to C30, C28 to C31, C29 to C32, C30 to C33, C31 to C34, C32 to C35, C41 to C45, C42 to C46, C2 to C5, C51 to C56, C52 to C57, C53 to C58, C55 to C60, C57 to C62, C4 to C7, C5 to C8, C6 to C9, DBG31 to DBG1, DBG32 to DBG2, DBG40 to DBG24, DBG41 to DBG25, DBG42 to DBG26, DBG43 to DBG27, DBG33 to DBG3, DBG34 to DBG4, DBG35 to DBG5, DBG1 to DBG6, IC5 to IC6, IC6 to IC8, IC7 to IC9, LED5 to LED4, LED4 to LED5, LED7 to LED6, LED6 to LED7, R6 to R10, R7 to R13, R9 to R29, R21 to R35, R20 to R36, R19 to R37, R18 to R38, R22 to R43, R34 to R49, R33 to R50, R32 to R51, R31 to R52, R35 to R53, R4 to R6
Connections:
- net /SWD Pad/FLASH renamed /SWD Pad/BOOT0
- C43 pad 1: Net-(T1-CT_1) -> Net-(J5-CRD)
- C54 pad 1: Net-(T2-CT_1) -> Net-(J6-CRD)
- FB2 pad 1: +3V3 -> /System Ethernet/3V3_ETH
- FB2 pad 2: Net-(T1-CT_1) -> Net-(J5-CRD)
- FB3 pad 1: +3V3 -> /External Ethernet/3V3_ETH
- FB3 pad 2: Net-(T2-CT_1) -> Net-(J6-CRD)
- IC1 pad 13: /Power Supply/PW_OK -> unconnected-(IC1-PC1-Pad13)
- IC1 pad 14: /Power Supply/PW_ON -> unconnected-(IC1-PC2-Pad14)
- IC1 pad 15: unconnected-(IC1-PC3-Pad15) -> /OLED Socket/SDI
- IC1 pad 20: /COM Bus Header/RTS -> unconnected-(IC1-PA1-Pad20)
- IC1 pad 21: /COM Bus Header/TX -> unconnected-(IC1-PA2-Pad21)
- IC1 pad 22: /COM Bus Header/RX -> /Microcontroller/SYSETH_XFRM_EN
- IC1 pad 29: /Microcontroller/SYSTEH_~{RST} -> /Microcontroller/SYSTEH_~{INT}
- IC1 pad 30: /Microcontroller/SYSTEH_~{INT} -> /Microcontroller/SYSTEH_~{RST}
- IC1 pad 31: unconnected-(IC1-PB2-Pad31) -> /SWD Pad/BOOT1
- IC1 pad 4: /External Ethernet/~{RST} -> /OLED Socket/~{RST}
- IC1 pad 41: /External Ethernet/SCK -> /COM Bus Header/TX
- IC1 pad 42: unconnected-(IC1-PB11-Pad42) -> /COM Bus Header/RX
- IC1 pad 46: /External Ethernet/CS -> unconnected-(IC1-PB12-Pad46)
- IC1 pad 47: unconnected-(IC1-PB13-Pad47) -> /COM Bus Header/CTS
- IC1 pad 48: /External Ethernet/SDO -> /COM Bus Header/RTS
- IC1 pad 49: /External Ethernet/SDI -> unconnected-(IC1-PB15-Pad49)
- IC1 pad 5: unconnected-(IC1-PC14-Pad5) -> /OLED Socket/DC
- IC1 pad 50: /Front Panel Client/PWR_ON -> unconnected-(IC1-PD8-Pad50)
- IC1 pad 51: /Front Panel Client/RESET -> unconnected-(IC1-PD9-Pad51)
- IC1 pad 68: unconnected-(IC1-PC8-Pad68) -> /Front Panel Client/PWR_ON
- IC1 pad 69: unconnected-(IC1-PC9-Pad69) -> /Front Panel Client/RESET
- IC1 pad 80: /OLED Socket/CS -> /External Ethernet/CS
- IC1 pad 81: /OLED Socket/SCK -> /External Ethernet/SCK
- IC1 pad 82: /OLED Socket/DC -> /External Ethernet/SDO
- IC1 pad 83: /OLED Socket/SDI -> /External Ethernet/SDI
- IC1 pad 84: /OLED Socket/~{RST} -> /External Ethernet/~{RST}
- IC1 pad 85: unconnected-(IC1-PD1-Pad85) -> /External Ethernet/~{INT}
- IC1 pad 86: unconnected-(IC1-PD2-Pad86) -> /External Ethernet/XFRM_EN
- IC1 pad 87: /COM Bus Header/CTS -> /OLED Socket/SCK
- IC1 pad 89: unconnected-(IC1-PD5-Pad89) -> /Power Supply/PW_OK
- IC1 pad 90: unconnected-(IC1-PD6-Pad90) -> /Power Supply/PW_ON
- IC1 pad 99: /External Ethernet/~{INT} -> /OLED Socket/CS
- IC4 pad 12: /System Ethernet/TPIN- -> /System Ethernet/ETH_TPIN-
- IC4 pad 13: /System Ethernet/TPIN+ -> /System Ethernet/ETH_TPIN+
- IC4 pad 16: /System Ethernet/TPOUT- -> /System Ethernet/ETH_TPOUT-
- IC4 pad 17: /System Ethernet/TPOUT+ -> /System Ethernet/ETH_TPOUT+
- IC6 pad 12: /External Ethernet/TPIN- -> /External Ethernet/ETH_TPIN-
- IC6 pad 13: /External Ethernet/TPIN+ -> /External Ethernet/ETH_TPIN+
- IC6 pad 16: /External Ethernet/TPOUT- -> /External Ethernet/ETH_TPOUT-
- IC6 pad 17: /External Ethernet/TPOUT+ -> /External Ethernet/ETH_TPOUT+
- J4 pad 24: GND -> /OLED Socket/D2
- J4 pad 25: GND -> /OLED Socket/D3
- J4 pad 26: GND -> /OLED Socket/D4
- J4 pad 27: GND -> /OLED Socket/D5
- J4 pad 28: GND -> /OLED Socket/D6
- J4 pad 29: GND -> /OLED Socket/D7
- J4 pad 7: unconnected-(J4-Pad7) -> Net-(J4-Pad7)
- J5 pad 1: /System Ethernet/TX+ -> /System Ethernet/ETH_TPOUT+
- J5 pad 11: Net-(J5-A_GREEN) -> +3V3
- J5 pad 12: GND -> Net-(J5-GLED_C)
- J5 pad 2: /System Ethernet/TX- -> Net-(J5-CRD)
- J5 pad 3: /System Ethernet/RX+ -> /System Ethernet/ETH_TPOUT-
- J5 pad 4: /System Ethernet/CT_45 -> /System Ethernet/ETH_TPIN+
- J5 pad 5: /System Ethernet/CT_45 -> Net-(J5-CRD)
- J5 pad 6: /System Ethernet/RX- -> /System Ethernet/ETH_TPIN-
- J5 pad 7: /System Ethernet/CT_78 -> unconnected-(J5-NC-Pad7)
- J5 pad 8: /System Ethernet/CT_78 -> Earth
- J6 pad 1: /External Ethernet/TX+ -> /External Ethernet/ETH_TPOUT+
- J6 pad 11: Net-(J6-A_GREEN) -> +3V3
- J6 pad 12: GND -> Net-(J6-GLED_C)
- J6 pad 2: /External Ethernet/TX- -> Net-(J6-CRD)
- J6 pad 3: /External Ethernet/RX+ -> /External Ethernet/ETH_TPOUT-
- J6 pad 4: /External Ethernet/CT_45 -> /External Ethernet/ETH_TPIN+
- J6 pad 5: /External Ethernet/CT_45 -> Net-(J6-CRD)
- J6 pad 6: /External Ethernet/RX- -> /External Ethernet/ETH_TPIN-
- J6 pad 7: /External Ethernet/CT_78 -> unconnected-(J6-NC-Pad7)
- J6 pad 8: /External Ethernet/CT_78 -> Earth
- J7 pad 1: /SWD Pad/VCC -> +3V3
- J7 pad 2: GND -> /SWD Pad/BOOT1
- LED1 pad 1: Net-(LED1-Pad1) -> GND
- LED1 pad 2: +3V3 -> Net-(LED1-Pad2)
- LED5 pad 1: GND -> Net-(LED5-Pad1)
- LED5 pad 2: Net-(LED4-Pad2) -> +3V3
- LED7 pad 1: GND -> Net-(LED7-Pad1)
- LED7 pad 2: Net-(LED6-Pad2) -> +3V3
- R14 pad 1: Net-(T1-CT_3) -> Net-(J4-Pad7)
- R14 pad 2: Net-(C35-Pad2) -> GND
- R15 pad 1: Net-(T1-CT_4) -> /OLED Socket/D2
- R15 pad 2: Net-(C35-Pad2) -> GND
- R16 pad 1: /System Ethernet/CT_45 -> /OLED Socket/D3
- R16 pad 2: Net-(C35-Pad2) -> GND
- R17 pad 1: /System Ethernet/CT_78 -> /OLED Socket/D4
- R17 pad 2: Net-(C35-Pad2) -> GND
- R27 pad 1: Net-(T2-CT_3) -> GND
- R27 pad 2: Net-(C45-Pad2) -> /Microcontroller/SYSETH_MISO
- R28 pad 1: Net-(T2-CT_4) -> GND
- R28 pad 2: Net-(C45-Pad2) -> /Microcontroller/SYSTEH_~{RST}
- R30 pad 1: /External Ethernet/CT_78 -> GND
- R30 pad 2: Net-(C45-Pad2) -> /Microcontroller/SYSETH_XFRM_EN
- R31 pad 1: /System Ethernet/TPOUT+ -> /System Ethernet/ETH_TPOUT+
- R31 pad 2: Net-(T1-CT_1) -> Net-(J5-CRD)
- R32 pad 1: /System Ethernet/TPOUT- -> /System Ethernet/ETH_TPOUT-
- R32 pad 2: Net-(T1-CT_1) -> Net-(J5-CRD)
- R33 pad 1: /System Ethernet/TPIN+ -> /System Ethernet/ETH_TPIN+
- R34 pad 1: /System Ethernet/TPIN- -> /System Ethernet/ETH_TPIN-
- R35 pad 1: Net-(LED4-Pad2) -> Net-(LED5-Pad1)
- R37 pad 1: Net-(J5-A_GREEN) -> Net-(J5-GLED_C)
- R45 pad 1: /External Ethernet/TPOUT+ -> /External Ethernet/ETH_TPOUT+
- R45 pad 2: Net-(T2-CT_1) -> Net-(J6-CRD)
- R46 pad 1: /External Ethernet/TPOUT- -> /External Ethernet/ETH_TPOUT-
- R46 pad 2: Net-(T2-CT_1) -> Net-(J6-CRD)
- R47 pad 1: /External Ethernet/TPIN+ -> /External Ethernet/ETH_TPIN+
- R48 pad 1: /External Ethernet/TPIN- -> /External Ethernet/ETH_TPIN-
- R49 pad 1: Net-(LED6-Pad2) -> Net-(LED7-Pad1)
- R51 pad 1: Net-(J6-A_GREEN) -> Net-(J6-GLED_C)
- R6 pad 2: Net-(LED1-Pad1) -> Net-(LED1-Pad2)
Routing:
- net GNDPWR: track 218.1 -> 0.00 mm, vias 8 -> 0
- net +5V: track 186.3 -> 0.00 mm, vias 5 -> 0
- net GND: track 161.2 -> 9.35 mm, vias 142 -> 6
- net +3V3: track 94.3 -> 0.00 mm, vias 38 -> 0
- net /SWD Pad/SWDIO: track 77.8 -> 0.00 mm, vias 2 -> 0
- net /OLED Socket/SCK: track 75.6 -> 0.00 mm
- net /Power Supply/PW_OK: track 72.3 -> 0.00 mm, vias 1 -> 0
- net /SWD Pad/SWCLK: track 71.5 -> 0.00 mm, vias 2 -> 0
- net /OLED Socket/~{RST}: track 69.2 -> 0.00 mm, vias 2 -> 0
- net /OLED Socket/DC: track 65.6 -> 0.00 mm, vias 2 -> 0
- net /OLED Socket/SDI: track 65.0 -> 0.00 mm
- net /Front Panel Client/HDD+: track 60.0 -> 0.00 mm, vias 1 -> 0
- net /OLED Socket/CS: track 60.0 -> 0.00 mm, vias 2 -> 0
- net /Front Panel Client/HDD-: track 58.3 -> 0.00 mm, vias 1 -> 0
- net /SWD Pad/BOOT0: track 57.2 -> 0.00 mm, vias 2 -> 0
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Other:
- board text removed: "0"
- board text removed: "0 mm"
- board text removed: "0.01 mm"
- board text removed: "0.0152 mm"
- board text removed: "0.02"
- board text removed: "0.035 mm"
- board text removed: "0.0900 mm / 0.0900 mm"
- board text removed: "0.1500 mm"
- board text removed: "0.2104 mm"
- board text removed: "1"
- board text removed: "1.065 mm"
- board text removed: "1.6062 mm"
- board text removed: "114.9000 mm x 65.4479 mm"
- board text removed: "3.3"
- board text removed: "4"
- board text removed: "4.5"
- board text removed: "B.Cu"
- board text removed: "B.Mask"
- board text removed: "B.Paste"
- board text removed: "B.Silkscreen"
- board text removed: "BOARD CHARACTERISTICS"
- board text removed: "Board Thickness:"
- board text removed: "Board overall dimensions:"
- board text removed: "Bottom Silk Screen"
- board text removed: "Bottom Solder Mask"
- board text removed: "Bottom Solder Paste"
- board text removed: "Castellated pads:"
- board text removed: "Color"
- board text removed: "Copper Finish:"
- board text removed: "Copper Layer Count:"
- board text removed: "Dielectric"
- board text removed: "ENIG"
- board text removed: "Edge card connectors:"
- board text removed: "Epsilon R"
- board text removed: "F.Cu"
- board text removed: "F.Mask"
- board text removed: "F.Paste"
- board text removed: "F.Silkscreen"
- board text removed: "FR4"
- board text removed: "Impedance Control:"
- board text removed: "In1.Cu"
- board text removed: "In2.Cu"
- board text removed: "JLC04161H-7628"
- board text removed: "Layer Name"
- board text removed: "Loss Tangent"
- board text removed: "Material"
- board text removed: "Min hole diameter:"
- board text removed: "Min track/spacing:"
- board text removed: "No"
- board text removed: "Not specified"
- board text removed: "Plated Board Edge:"
- board text removed: "Thickness (mm)"
- board text removed: "Top Silk Screen"
- board text removed: "Top Solder Mask"
- board text removed: "Top Solder Paste"
- board text removed: "Type"
- board text removed: "copper"
- board text removed: "core"
- board text removed: "prepreg"

Commit message: ethernet ports wired up
Parts:
- removed C3: 1nF 5kV, SamacSys_Parts:CAPC4620X220N
- removed DBG1, DBG10, DBG11, DBG12, DBG13, DBG14, DBG15, DBG16, DBG17, DBG18, DBG19, DBG2, DBG20, DBG21, DBG22, DBG23, DBG24, DBG25, DBG26, DBG27, DBG28, DBG29, DBG3, DBG30, DBG31, DBG32, DBG4, DBG5, DBG6, DBG7, DBG8, DBG9: ~, Oro Footprints:DebugPin
- C1, C2: value 1nF 5kV -> 1nF 3kV
- FB2, FB3: moved to F.Cu
- moved R39 181.2 mm to (223.6, 77.1)
- moved R40 181.2 mm to (223.6, 79.3)
- moved R41 181.2 mm to (223.6, 81.4)
- moved R42 181.2 mm to (223.6, 83.6)
- moved R44 181.2 mm to (223.6, 85.7)
- moved IC7 169.1 mm to (195.1, 84.5), turned to 90 degrees
- moved C52 165.4 mm to (194.6, 81.3), turned to 180 degrees
- moved C55 161.9 mm to (192.4, 91.2)
- moved C2 134.0 mm to (175.8, 92.1), turned to 90 degrees
- moved C41 96.2 mm to (122.8, 90.4), turned to -90 degrees
- moved C44 92.1 mm to (118.6, 90.7), turned to 90 degrees
- moved C53 78.0 mm to (179.5, 91.6), turned to 180 degrees
- moved R48 76.5 mm to (181.7, 91.6), turned to 180 degrees
- moved R46 75.6 mm to (186.2, 91.6), turned to 180 degrees
- moved R47 72.7 mm to (183.8, 91.6), turned to 0 degrees
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Connections:
- C1 pad 1: GNDPWR -> Earth
- C2 pad 1: GNDPWR -> Earth
- C43 pad 1: Net-(J5-CRD) -> Net-(J5-CTD)
- C44 pad 1: Net-(J5-CRD) -> Net-(J5-CTD)
- C54 pad 1: Net-(J6-CRD) -> Net-(J6-CTD)
- C55 pad 1: Net-(J6-CRD) -> Net-(J6-CTD)
- D1 pad 2: GNDPWR -> GND
- D2 pad 2: GNDPWR -> GND
- FB2 pad 2: Net-(J5-CRD) -> Net-(J5-CTD)
- FB3 pad 2: Net-(J6-CRD) -> Net-(J6-CTD)
- H1 pad 1: GNDPWR -> (no net)
- H2 pad 1: GNDPWR -> (no net)
- H3 pad 1: GNDPWR -> (no net)
- H4 pad 1: GND -> (no net)
- J5 pad 1: /System Ethernet/ETH_TPOUT+ -> /System Ethernet/ETH_TPOUT-
- J5 pad 2: Net-(J5-CRD) -> Net-(J5-CTD)
- J5 pad 3: /System Ethernet/ETH_TPOUT- -> /System Ethernet/ETH_TPOUT+
- J5 pad 4: /System Ethernet/ETH_TPIN+ -> /System Ethernet/ETH_TPIN-
- J5 pad 5: Net-(J5-CRD) -> unconnected-(J5-CRD-Pad5)
- J5 pad 6: /System Ethernet/ETH_TPIN- -> /System Ethernet/ETH_TPIN+
- J6 pad 1: /External Ethernet/ETH_TPOUT+ -> /External Ethernet/ETH_TPOUT-
- J6 pad 2: Net-(J6-CRD) -> Net-(J6-CTD)
- J6 pad 3: /External Ethernet/ETH_TPOUT- -> /External Ethernet/ETH_TPOUT+
- J6 pad 4: /External Ethernet/ETH_TPIN+ -> /External Ethernet/ETH_TPIN-
- J6 pad 5: Net-(J6-CRD) -> unconnected-(J6-CRD-Pad5)
- J6 pad 6: /External Ethernet/ETH_TPIN- -> /External Ethernet/ETH_TPIN+
- R31 pad 1: /System Ethernet/ETH_TPOUT+ -> /System Ethernet/ETH_TPOUT-
- R31 pad 2: Net-(J5-CRD) -> Net-(J5-CTD)
- R32 pad 1: /System Ethernet/ETH_TPOUT- -> /System Ethernet/ETH_TPOUT+
- R32 pad 2: Net-(J5-CRD) -> Net-(J5-CTD)
- R33 pad 1: /System Ethernet/ETH_TPIN+ -> /System Ethernet/ETH_TPIN-
- R34 pad 1: /System Ethernet/ETH_TPIN- -> /System Ethernet/ETH_TPIN+
- R45 pad 1: /External Ethernet/ETH_TPOUT+ -> /External Ethernet/ETH_TPOUT-
- R45 pad 2: Net-(J6-CRD) -> Net-(J6-CTD)
- R46 pad 1: /External Ethernet/ETH_TPOUT- -> /External Ethernet/ETH_TPOUT+
- R46 pad 2: Net-(J6-CRD) -> Net-(J6-CTD)
- R47 pad 1: /External Ethernet/ETH_TPIN+ -> /External Ethernet/ETH_TPIN-
- R48 pad 1: /External Ethernet/ETH_TPIN- -> /External Ethernet/ETH_TPIN+
Routing:
- net GND: track 9.35 -> 99.3 mm, vias 6 -> 34
- net +3V3: track 0.00 -> 70.4 mm, vias 0 -> 15
- net Net-(J5-GLED_C): track 0.00 -> 26.9 mm
- net Net-(J6-YLED_A): track 0.00 -> 24.9 mm
- net Earth: track 0.00 -> 23.5 mm
- net Net-(J6-CTD): track 0.00 -> 19.8 mm, vias 0 -> 2
- net Net-(LED5-Pad1): track 0.00 -> 18.2 mm, vias 0 -> 2
- net Net-(J5-CTD): track 0.00 -> 17.1 mm, vias 0 -> 2
- net /External Ethernet/ETH_TPOUT+: track 0.00 -> 14.8 mm
- net /External Ethernet/ETH_TPOUT-: track 0.00 -> 14.8 mm
- net /System Ethernet/ETH_TPOUT-: track 0.00 -> 14.5 mm
- net /System Ethernet/ETH_TPOUT+: track 0.00 -> 14.5 mm
- net /System Ethernet/ETH_TPIN-: track 0.00 -> 13.7 mm
- net /System Ethernet/ETH_TPIN+: track 0.00 -> 13.7 mm
- net Net-(J5-YLED_A): track 0.00 -> 13.5 mm
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
Commit message: don't use global earth power symbol for ethernet earths
Connections:
- C1 pad 1: Earth -> /System Ethernet/RJ_EARTH
- C2 pad 1: Earth -> /External Ethernet/RJ_EARTH
- J5 pad 14: Earth -> /System Ethernet/RJ_EARTH
- J5 pad 8: Earth -> /System Ethernet/RJ_EARTH
- J6 pad 14: Earth -> /External Ethernet/RJ_EARTH
- J6 pad 8: Earth -> /External Ethernet/RJ_EARTH
Routing:
- net Earth: track 23.5 -> 0.00 mm
- net /System Ethernet/RJ_EARTH: track 0.00 -> 11.8 mm
- net /External Ethernet/RJ_EARTH: track 0.00 -> 11.7 mm

Commit message: preliminary component placement for rev5
Parts:
- moved R39 49.9 mm to (174.0, 82.3)
- moved R40 49.8 mm to (174.0, 83.4)
- moved R41 49.8 mm to (174.0, 84.6)
- moved R42 49.7 mm to (174.0, 85.7)
- moved R44 49.7 mm to (174.0, 86.9)
Changed lines of the file:
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@@
   )
   (footprint "SamacSys_Parts:RESC1005X40N" (layer "F.Cu")
-    (at 223.647 83.557)
+    (at 173.99 85.725)
     (descr "1E(0402)")
     (tags "Resistor")
@@
   )
   (footprint "SamacSys_Parts:RESC1005X40N" (layer "F.Cu")
-    (at 223.647 85.707)
+    (at 173.99 86.868)
     (descr "1E(0402)")
     (tags "Resistor")
@@
   )
   (footprint "SamacSys_Parts:RESC1005X40N" (layer "F.Cu")
-    (at 223.647 77.107)
+    (at 173.99 82.314)
     (descr "1E(0402)")
     (tags "Resistor")
@@
   )
   (footprint "SamacSys_Parts:RESC1005X40N" (layer "F.Cu")
-    (at 223.647 81.407)
+    (at 173.99 84.582)
     (descr "1E(0402)")
     (tags "Resistor")
@@
   )
   (footprint "SamacSys_Parts:RESC1005X40N" (layer "F.Cu")
-    (at 223.647 79.257)
+    (at 173.99 83.439)
     (descr "1E(0402)")
     (tags "Resistor")

Commit message: most power routing completed
Parts:
- moved R13 1.52 mm to (163.4, 102.5)
- moved R15 1.27 mm to (103.9, 51.3)
- moved R17 1.27 mm to (105.2, 51.3)
- moved R10 0.89 mm to (161.0, 102.5)
- moved C61 0.71 mm to (164.5, 69.2)
- moved C62 0.71 mm to (163.2, 69.2)
- moved C12 0.68 mm to (136.5, 74.7)
- moved C8 0.57 mm to (135.3, 93.7)
- moved C14 0.42 mm to (137.0, 94.4), turned to -45 degrees
- moved C19 0.37 mm to (132.5, 78.7)
- moved C20 0.37 mm to (131.6, 77.9)
Connections:
- S2 pad 2: +5V -> /Power Supply/5VSB
- S2 pad 4: /Power Supply/5VSB -> +5V
Routing:
- net +5V: track 0.00 -> 162.8 mm, vias 0 -> 2
- net GND: track 99.3 -> 176.8 mm, vias 34 -> 64
- net +3V3: track 70.4 -> 135.3 mm, vias 15 -> 39
- net /OLED Socket/+12V: track 0.00 -> 36.1 mm, vias 0 -> 3
- net Net-(Q1-Pad3): track 0.00 -> 33.9 mm, vias 0 -> 1
- net /Power Supply/5VSB: track 0.00 -> 22.8 mm
- net /Power Supply/PSU_ON: track 0.00 -> 18.1 mm
- net /OLED Socket/D7: track 0.00 -> 15.0 mm
- net /OLED Socket/D5: track 0.00 -> 13.9 mm
- net /OLED Socket/D3: track 0.00 -> 12.9 mm
- net /OLED Socket/DC: track 0.00 -> 10.4 mm
- net /OLED Socket/CS: track 0.00 -> 9.36 mm
- net Net-(IC3-OUT): track 0.00 -> 9.08 mm, vias 0 -> 1
- net /OLED Socket/~{RST}: track 0.00 -> 8.27 mm
- net /SWD Pad/BOOT1: track 0.00 -> 6.49 mm
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