File: pcb/link-x86-obt/front-panel-client.kicad_sch (KiCad schematic)
At the start: 9 parts, among them IC16 PMV20ENR, IC18 PMV20ENR, J10 67996-408HLF

Commit message: add P-channel mosfet to 5VSB line
Parts:
- renumbered J10 to J3
