File: pcb/link/link.kicad_sch (KiCad schematic)
At the start: 91 parts, among them J1 STLINK-V3MINIE, J11 68021-204HLF, J13 68021-204HLF, J16 68021-204HLF, J18 68021-204HLF, J5 68021-204HLF, Q2 PMV20ENR, Q3 PMV20ENR, SW1 TL6400AF160QJ, U1 STM32F479VGT6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

Commit message: remove 3V3VREF TP (and upgrade to kicad 10) (closes #105)
Parts:
- TP11, TP12: value ~ -> (none)
