File: pcb/link/power.kicad_sch (KiCad schematic)
At the start: 45 parts, among them J3 SACC-DSIV-M12MS-5CON-L180, J7 USB4105-GF-A, Q1 PMV20ENR, U12 LM1085ISX-3.3/NOPB, U13 INA226AIDGSR, U9 LTC4415EMSE#TRPBF

Commit message: add MQTT stats system
Parts:
- U9: value LTC4415EMSE#TRPBF -> LTC4415EMSE
Changed lines of the file:
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@@
 			)
 		)
-		(property "Value" "LTC4415EMSE#TRPBF"
+		(property "Value" "LTC4415EMSE"
 			(at 109.22 36.239 0)
 			(show_name no)
